File: AR20_ACM/ACM_pcb/KiCAD/ACM_Y2020V0.1/ACM_Y2020V0.1.sch (KiCad schematic (older format))
At the start: 23 parts, among them J1 TC2030-MCP-NL, J2 Conn_02x15_Odd_Even, Q1 Q_PMOS_DGS, U1 ATmega328PB-AU, U2 MCP25625-x-SS, U3 SPX3819M5-L-5-0, Y1 16.0Mhz

Commit message: Changelog for 29.07.2019
Connections:
- net U-Pin15 is gone; now on net MISO: J2.15 (Pin_15)
- net U-Pin17 is gone; now on net MOSI: J2.17 (Pin_17)
- net +12V: now also J2.29 (Pin_29); no longer J2.1 (Pin_1)
- net +5V: now also J2.27 (Pin_27); no longer J2.3 (Pin_3)
- net Reset: no longer J2.10 (Pin_10)
- net U-Pin25: no longer names the net of J2.25 (Pin_25)
- net U-Pin27 renamed U-Pin3
- net U-Pin3: now also J2.3 (Pin_3); no longer J2.27 (Pin_27)
- net U-Pin29 renamed U-Pin1
- net U-Pin1: now also J2.1 (Pin_1); no longer J2.29 (Pin_29)
Other:
- moved on the sheet: Y1
Changed lines of the file:
@@
 Text HLabel 2775 5075 2    50   Input ~ 0
 SCK
-Text HLabel 2775 4975 2    50   Input ~ 0
+Text HLabel 2800 4950 2    25   Input ~ 0
 MISO
-Text HLabel 2775 4875 2    50   Input ~ 0
+Text HLabel 2800 4850 2    25   Input ~ 0
 MOSI
 Text HLabel 3075 1500 2    50   Input ~ 0
@@
 L Device:Resonator_Small Y1
 U 1 1 5D3C125F
-P 3200 5225
-F 0 "Y1" V 3475 5200 50  0000 C CNN
-F 1 "16.0Mhz" V 3400 5200 50  0000 C CNN
-F 2 "CSTNE16M0V530000R0:CSTNE16M0V530000R0" H 3175 5225 50  0001 C CNN
-F 3 "~" H 3175 5225 50  0001 C CNN
-	1    3200 5225
+P 3700 5250
+F 0 "Y1" V 3975 5225 50  0000 C CNN
+F 1 "16.0Mhz" V 3900 5225 50  0000 C CNN
+F 2 "CSTNE16M0V530000R0:CSTNE16M0V530000R0" H 3675 5250 50  0001 C CNN
+F 3 "~" H 3675 5250 50  0001 C CNN
+	1    3700 5250
 	0    -1   -1   0
 $EndComp
@@
 L power:GND #PWR0107
 U 1 1 5D3C307D
-P 3450 5275
-F 0 "#PWR0107" H 3450 5025 50  0001 C CNN
-F 1 "GND" H 3455 5102 50  0000 C CNN
-F 2 "" H 3450 5275 50  0001 C CNN
-F 3 "" H 3450 5275 50  0001 C CNN
-	1    3450 5275
-	1    0    0    -1
-$EndComp
-Wire Wire Line
-	3400 5225 3450 5225
-Wire Wire Line
-	3450 5225 3450 5275
+P 3950 5300
+F 0 "#PWR0107" H 3950 5050 50  0001 C CNN
+F 1 "GND" H 3955 5127 50  0000 C CNN
+F 2 "" H 3950 5300 50  0001 C CNN
+F 3 "" H 3950 5300 50  0001 C CNN
+	1    3950 5300
+	1    0    0    -1
+$EndComp
+Wire Wire Line
+	3900 5250 3950 5250
+Wire Wire Line
+	3950 5250 3950 5300
 $Comp
 L Device:R R1
@@
 Close as possible to MCP-chip
 Wire Wire Line
-	2775 5175 3000 5175
-Wire Wire Line
-	3000 5175 3000 5125
-Wire Wire Line
-	3000 5125 3100 5125
-Wire Wire Line
-	3100 5325 3000 5325
-Wire Wire Line
-	3000 5325 3000 5275
-Wire Wire Line
-	3000 5275 2775 5275
+	3500 5150 3600 5150
+Wire Wire Line
+	3600 5350 3500 5350
 Text Notes 9275 2925 0    79   ~ 16
 CAN MCU
@@
 L power:+12V #PWR0121
 U 1 1 5D3DBA57
-P 5150 1075
-F 0 "#PWR0121" H 5150 925 50  0001 C CNN
-F 1 "+12V" H 5165 1248 50  0000 C CNN
-F 2 "" H 5150 1075 50  0001 C CNN
-F 3 "" H 5150 1075 50  0001 C CNN
-	1    5150 1075
-	1    0    0    -1
-$EndComp
-Wire Wire Line
-	5150 1075 5150 1175
-Wire Wire Line
-	5150 1175 5400 1175
+P 5475 2850
+F 0 "#PWR0121" H 5475 2700 50  0001 C CNN
+F 1 "+12V" H 5490 3023 50  0000 C CNN
+F 2 "" H 5475 2850 50  0001 C CNN
+F 3 "" H 5475 2850 50  0001 C CNN
+	1    5475 2850
+	1    0    0    -1
+$EndComp
 $Comp
 L power:+5V #PWR0122
 U 1 1 5D3DED37
-P 4950 1075
-F 0 "#PWR0122" H 4950 925 50  0001 C CNN
-F 1 "+5V" H 4965 1248 50  0000 C CNN
-F 2 "" H 4950 1075 50  0001 C CNN
-F 3 "" H 4950 1075 50  0001 C CNN
-	1    4950 1075
-	1    0    0    -1
-$EndComp
-Wire Wire Line
-	4950 1075 4950 1275
+P 5075 2825
+F 0 "#PWR0122" H 5075 2675 50  0001 C CNN
+F 1 "+5V" H 5090 2998 50  0000 C CNN
+F 2 "" H 5075 2825 50  0001 C CNN
+F 3 "" H 5075 2825 50  0001 C CNN
+	1    5075 2825
+	1    0    0    -1
+$EndComp
 $Comp
 L power:GND #PWR0123
@@
 Wire Wire Line
 	10175 1450 10175 1375
-Text HLabel 2775 6775 2    50   Input ~ 0
+Text HLabel 2800 6750 2    25   Input ~ 0
 GREEN_LED
-Text HLabel 2850 4675 2    50   Input ~ 0
+Text HLabel 2850 4675 2    25   Input ~ 0
 RED_LED
-Text HLabel 2850 4800 2    50   Input ~ 0
+Text HLabel 2850 4800 2    25   Input ~ 0
 BLUE_LED
 Text HLabel 5900 1475 2    50   Input ~ 0
@@
 	1    0    0    -1
 $EndComp
-Text HLabel 5900 1575 2    50   Input ~ 0
+Text HLabel 5925 1575 2    50   Input ~ 0
 U-Pin10
 Text HLabel 5900 1675 2    50   Input ~ 0
@@
 	5975 5300 6675 5300
 Connection ~ 5975 5300
-Wire Wire Line
-	4950 1275 5400 1275
 Wire Wire Line
 	5900 1875 6025 1875
@@
 Text HLabel 5400 2275 0    50   Input ~ 0
 U-Pin23
-Text HLabel 5400 2375 0    50   Input ~ 0
+Text HLabel 5350 2375 0    50   Input ~ 0
 U-Pin25
-Text HLabel 5400 2475 0    50   Input ~ 0
-U-Pin27
-Text HLabel 5400 2575 0    50   Input ~ 0
-U-Pin29
+Text HLabel 5400 1175 0    50   Input ~ 0
+U-Pin1
+Text HLabel 5400 1275 0    50   Input ~ 0
+U-Pin3
 Text HLabel 5900 1375 2    50   Input ~ 0
 U-Pin6
@@
 Text HLabel 1575 6575 0    50   Input ~ 0
 U-Pin9
-Text HLabel 2775 6875 2    50   Input ~ 0
-U-Pin23
 Text HLabel 2775 6675 2    50   Input ~ 0
 U-Pin22
@@
 Text HLabel 2775 6275 2    50   Input ~ 0
 U-Pin12
-Text HLabel 3450 6125 2    50   Input ~ 0
+Text HLabel 3475 6125 2    50   Input ~ 0
 U-Pin10
 Wire Wire Line
@@
 Text HLabel 2775 5475 2    50   Input ~ 0
 U-Pin7
-Text HLabel 2850 4625 2    50   Input ~ 0
+Text HLabel 2850 4625 2    25   Input ~ 0
 U-Pin21
-Text HLabel 2850 4750 2    50   Input ~ 0
+Text HLabel 2850 4750 2    25   Input ~ 0
 U-Pin19
 Wire Wire Line
@@
 Connection ~ 2800 4775
 Text HLabel 10775 3900 2    50   Input ~ 0
-U-Pin27
+U-Pin3
 Text HLabel 10775 4200 2    50   Input ~ 0
-U-Pin29
+U-Pin1
+Wire Wire Line
+	5400 2575 5300 2575
+Wire Wire Line
+	5300 2575 5300 2900
+Wire Wire Line
+	5300 2900 5475 2900
+Wire Wire Line
+	5475 2900 5475 2850
+Wire Wire Line
+	5400 2475 5250 2475
+Wire Wire Line
+	5250 2475 5250 2900
+Wire Wire Line
+	5250 2900 5075 2900
+Wire Wire Line
+	5075 2900 5075 2825
+Wire Wire Line
+	2775 5175 3500 5175
+Wire Wire Line
+	3500 5175 3500 5150
+Wire Wire Line
+	3500 5350 3500 5275
+Wire Wire Line
+	3500 5275 2775 5275
+Text HLabel 2800 4900 2    25   Input ~ 0
+U-Pin17
+Text HLabel 2800 5000 2    25   Input ~ 0
+U-Pin15
+Wire Wire Line
+	2800 5000 2775 5000
+Wire Wire Line
+	2775 5000 2775 4975
+Wire Wire Line
+	2775 4975 2775 4950
+Wire Wire Line
+	2775 4950 2800 4950
+Connection ~ 2775 4975
+Wire Wire Line
+	2800 4900 2775 4900
+Wire Wire Line
+	2775 4900 2775 4875
+Wire Wire Line
+	2775 4875 2775 4850
+Wire Wire Line
+	2775 4850 2800 4850
+Connection ~ 2775 4875
+Text HLabel 2775 6875 2    50   Input ~ 0
+U-Pin23
+Wire Wire Line
+	2775 6775 2775 6800
+Wire Wire Line
+	2775 6800 2800 6800
+Wire Wire Line
+	2775 6775 2775 6750
+Wire Wire Line
+	2775 6750 2800 6750
+Connection ~ 2775 6775
+Text HLabel 2800 6800 2    25   Input ~ 0
+U-Pin25
 $EndSCHEMATC

Commit message: Changelog for 29.07.2019
Parts:
- added C6: 100nF, Capacitor_SMD:C_0402_1005Metric, symbol Device:C_Small
- added L1: 10uH, Inductor_SMD:L_0603_1608Metric, symbol Device:L_Small
Connections:
- net U-Pin13 is gone; now on net SCK: J2.13 (Pin_13)
- net +5V: now also L1.2; no longer U1.20 (AREF)
- net GND: now also C6.1
- net GREEN_LED: now also J2.25 (Pin_25)
- net Reset: now also J2.10 (Pin_10)
- new net: C6.2, L1.1, U1.20 (AREF)
- no-connect marks 0 -> 1
Other:
- note added: "AVCC Lavpass filter"
Changed lines of the file:
@@
 Text HLabel 2775 5075 2    50   Input ~ 0
 SCK
-Text HLabel 2800 4950 2    25   Input ~ 0
+Text HLabel 2850 4975 2    50   Input ~ 0
 MISO
-Text HLabel 2800 4850 2    25   Input ~ 0
+Text HLabel 2850 4875 2    50   Input ~ 0
 MOSI
 Text HLabel 3075 1500 2    50   Input ~ 0
@@
 	2175 4125 2175 4275
 Connection ~ 2175 4275
-Wire Wire Line
-	1575 4575 1575 4275
-Wire Wire Line
-	1575 4275 2175 4275
 $Comp
 L Device:C C1
@@
 	1    0    0    -1
 $EndComp
-Text HLabel 3450 6050 2    50   Input ~ 0
+Text HLabel 3450 6075 2    50   Input ~ 0
 Reset
 $Comp
@@
 Wire Wire Line
 	10175 1450 10175 1375
-Text HLabel 2800 6750 2    25   Input ~ 0
+Text HLabel 2775 6775 2    50   Input ~ 0
 GREEN_LED
-Text HLabel 2850 4675 2    25   Input ~ 0
+Text HLabel 2850 4675 2    50   Input ~ 0
 RED_LED
-Text HLabel 2850 4800 2    25   Input ~ 0
+Text HLabel 2875 4775 2    50   Input ~ 0
 BLUE_LED
-Text HLabel 5900 1475 2    50   Input ~ 0
-U-Pin8
 $Comp
 L power:GND #PWR0120
@@
 	1    0    0    -1
 $EndComp
-Text HLabel 5925 1575 2    50   Input ~ 0
-U-Pin10
 Text HLabel 5900 1675 2    50   Input ~ 0
 U-Pin12
@@
 Text HLabel 5400 1675 0    50   Input ~ 0
 U-Pin11
-Text HLabel 5400 1775 0    50   Input ~ 0
-U-Pin13
-Text HLabel 5400 1875 0    50   Input ~ 0
-U-Pin15
-Text HLabel 5400 1975 0    50   Input ~ 0
-U-Pin17
-Text HLabel 5400 2075 0    50   Input ~ 0
-U-Pin19
-Text HLabel 5400 2175 0    50   Input ~ 0
-U-Pin21
-Text HLabel 5400 2275 0    50   Input ~ 0
-U-Pin23
-Text HLabel 5350 2375 0    50   Input ~ 0
-U-Pin25
 Text HLabel 5400 1175 0    50   Input ~ 0
 U-Pin1
@@
 Text HLabel 2775 6275 2    50   Input ~ 0
 U-Pin12
-Text HLabel 3475 6125 2    50   Input ~ 0
-U-Pin10
-Wire Wire Line
-	3450 6125 3275 6125
-Wire Wire Line
-	3275 6125 3275 6075
-Wire Wire Line
-	3275 6075 3375 6075
-Wire Wire Line
-	3375 6075 3375 6050
-Wire Wire Line
-	3375 6050 3450 6050
 Connection ~ 3275 6075
 Wire Wire Line
@@
 Text HLabel 2775 5475 2    50   Input ~ 0
 U-Pin7
-Text HLabel 2850 4625 2    25   Input ~ 0
-U-Pin21
-Text HLabel 2850 4750 2    25   Input ~ 0
-U-Pin19
-Wire Wire Line
-	2775 4675 2800 4675
-Wire Wire Line
-	2800 4675 2800 4625
-Wire Wire Line
-	2800 4625 2850 4625
-Wire Wire Line
-	2850 4675 2800 4675
-Connection ~ 2800 4675
-Wire Wire Line
-	2775 4775 2800 4775
-Wire Wire Line
-	2800 4775 2800 4750
-Wire Wire Line
-	2800 4750 2850 4750
-Wire Wire Line
-	2850 4800 2800 4800
-Wire Wire Line
-	2800 4800 2800 4775
-Connection ~ 2800 4775
 Text HLabel 10775 3900 2    50   Input ~ 0
 U-Pin3
@@
 Wire Wire Line
 	3500 5275 2775 5275
-Text HLabel 2800 4900 2    25   Input ~ 0
-U-Pin17
-Text HLabel 2800 5000 2    25   Input ~ 0
-U-Pin15
-Wire Wire Line
-	2800 5000 2775 5000
-Wire Wire Line
-	2775 5000 2775 4975
-Wire Wire Line
-	2775 4975 2775 4950
-Wire Wire Line
-	2775 4950 2800 4950
-Connection ~ 2775 4975
-Wire Wire Line
-	2800 4900 2775 4900
-Wire Wire Line
-	2775 4900 2775 4875
-Wire Wire Line
-	2775 4875 2775 4850
-Wire Wire Line
-	2775 4850 2800 4850
-Connection ~ 2775 4875
 Text HLabel 2775 6875 2    50   Input ~ 0
 U-Pin23
-Wire Wire Line
-	2775 6775 2775 6800
-Wire Wire Line
-	2775 6800 2800 6800
-Wire Wire Line
-	2775 6775 2775 6750
-Wire Wire Line
-	2775 6750 2800 6750
-Connection ~ 2775 6775
-Text HLabel 2800 6800 2    25   Input ~ 0
-U-Pin25
+Text HLabel 5900 1575 2    50   Input ~ 0
+Reset
+Text HLabel 5900 1475 2    50   Input ~ 0
+U-Pin8
+Wire Wire Line
+	3275 6075 3450 6075
+Text HLabel 5400 1775 0    50   Input ~ 0
+SCK
+Wire Wire Line
+	2775 4675 2850 4675
+Wire Wire Line
+	2775 4775 2875 4775
+Wire Wire Line
+	2775 4875 2850 4875
+Wire Wire Line
+	2775 4975 2850 4975
+Text HLabel 5400 1875 0    50   Input ~ 0
+MISO
+Text HLabel 5400 1975 0    50   Input ~ 0
+MOSI
+Text HLabel 5400 2075 0    50   Input ~ 0
+BLUE_LED
+Text HLabel 5400 2175 0    50   Input ~ 0
+RED_LED
+Text HLabel 5400 2375 0    50   Input ~ 0
+GREEN_LED
+Text HLabel 5400 2275 0    50   Input ~ 0
+U-Pin23
+$Comp
+L Device:C_Small C6
+U 1 1 5D42F0C6
+P 1375 4675
+F 0 "C6" H 1283 4629 50  0000 R CNN
+F 1 "100nF" H 1283 4720 50  0000 R CNN
+F 2 "Capacitor_SMD:C_0402_1005Metric" H 1375 4675 50  0001 C CNN
+F 3 "http://www.farnell.com/datasheets/2620235.pdf?_ga=2.91386842.1939358490.1564414725-1415930916.1560114588&_gac=1.191516504.1564075292.CjwKCAjwpuXpBRAAEiwAyRRPgXwHZ1wF4xXBoNI_FJEvoVORJn7NbJB9jjbidsg8_qDnlLi_44u6wRoCV2MQAvD_BwE" H 1375 4675 50  0001 C CNN
+F 4 "https://no.farnell.com/vishay/vj0402y104kxjcw1bc/cap-0-1-f-16v-10-x7r-0402/dp/2896349?categoryId=700000005423&ddkey=https%3ASearch" H 1375 4675 50  0001 C CNN "Farnell"
+	1    1375 4675
+	-1   0    0    1
+$EndComp
+$Comp
+L power:GND #PWR0126
+U 1 1 5D431A06
+P 1375 4775
+F 0 "#PWR0126" H 1375 4525 50  0001 C CNN
+F 1 "GND" H 1380 4602 50  0000 C CNN
+F 2 "" H 1375 4775 50  0001 C CNN
+F 3 "" H 1375 4775 50  0001 C CNN
+	1    1375 4775
+	1    0    0    -1
+$EndComp
+NoConn ~ 1575 4575
+Wire Wire Line
+	1575 4575 1375 4575
+$Comp
+L Device:L_Small L1
+U 1 1 5D438986
+P 1625 4275
+F 0 "L1" V 1810 4275 50  0000 C CNN
+F 1 "10uH" V 1719 4275 50  0000 C CNN
+F 2 "Inductor_SMD:L_0603_1608Metric" H 1625 4275 50  0001 C CNN
+F 3 "http://www.farnell.com/datasheets/2761194.pdf?_ga=2.11278196.1939358490.1564414725-1415930916.1560114588&_gac=1.224087785.1564075292.CjwKCAjwpuXpBRAAEiwAyRRPgXwHZ1wF4xXBoNI_FJEvoVORJn7NbJB9jjbidsg8_qDnlLi_44u6wRoCV2MQAvD_BwE" H 1625 4275 50  0001 C CNN
+F 4 "https://no.farnell.com/kemet/l0603b100kpwft/inductor-10uh-0-2a-10-shielded/dp/2846740?sf=471%2C479%2C722&pf=110197189%2C113816526&krypto=wdlyXzEHzoNyTqp1ZIDmJKKAdm%2FeQwQzUV5II%2F3l7MkJePe%2BfKfknh2CgwpSUiLpJgcdHpbeKKQNs27Pjdo2jRSMMeJV4ksckB9bvQgjSQLUlPN%2F8kNke0kS%2F7e9zwpUlVUEfkQZfvA32jXqBxbhPFTsaDHlf4CUrJJagmXsEZ8VqOHUewBKNAKNFz24oGypoERTJ7jtqvZrwEWMlQvWyq%2Bkwmf5TKuw%2FM%2BKpLr8e4C3KwvQzXks9QHUZqIDOurzBMeJRKKPAU2Cop7koNP9ascTJrJphD%2BAV67YaEOEisxTmSVrp%2B67slUES2yOj2r0jG%2FjibhBGhVavKNC56O75cqVYQbb%2FzpPpCew%2FioTTozg98St7w8tL1P3vgWlxcp9fXPTAvmhLZb0EWKDlkueZvXeB%2BDmx2m%2Bgg2NUCj%2B32Vew0Ws%2Fp6lWVNU3dPlVFc63F7hbMfjDTGxBOc%2FTjp%2BEpGgO5R3SgaiwgWL%2FEzcIPG77sO%2BSCxcOvYq855M1ooR73PAfV3tiAYDIUbGLskav3MdSmjuyNqhqqbt%2BOW4eFTyio9upZ2rzvhqMgL3sNOXsdxFy1zMxFPE3g96cCOrVv90G0gTi%2F%2BC%2FdnWQWjMuJxMBWfEU2HHYGwtkhlbKhm5hV9S8DwwUUZcwx1JiZnZamPheGla%2Bghidf0HZ8WWxV%2FZExu%2FEr5aHjgV2fqrh1OcraGwEWPJLI6RdzosXCLSFOhkqDrGV9DxowzbxfooPoxlTzOSyLsnbWIT17I0hyUR%2FUyhF1bZOkUlY5KHF4WC0%2FbJ9%2BzlJwjY4u7qKhK0yzhBuCaJ77Bam5AzM08s%2FpYWr6zrlyjBCSGnVhMN0I8PxJsDcwrWO2QJOr0YaYUp3%2Bd1PSdPLPd0sABhGIfBAK%2FOfum4DMlifVQQts0%2F96wD9fet0PaV%2FTtf9s6BYt5%2FBFQSMob%2BZGKKrgc9rMAJ9wxKDeE2Y889JIh%2B0YE%2BrwzXRKQuGWIafhnxV8wkZxbM58FYqLYx8eZktu%2BsU%2BVMemuzC4EN0HGNIKpgVg363m4p8X0dNuuzk%2BIUSFGfWRr1h6fr%2FqKqcypB9dtMhW7gcYn5zLHTgE%2FS6cDRyKc74Qk7UiFSfB88IVhlUJSnF%2FuykwCYCPaUZpUg948Hp96p63d2FVKvr7vS8st4gcAR82WvRf69x9MDDjo%2BVGlNimRBQ3PVcyLBEQREozehuM5DjpfvSQwnm6bpggqkcR%2BFvgnfPG4tBc09ZsH9XCRRtcz9yyGKh5p6ROjbX%2FluOlj1sBzT%2Fk3eFbosFAMdN8nGXoaNq7xt9rXB7zNydT3EBLm0Xr7weln4LIWcz0Vim8f93f0YRlpFhJsEugj4D%2BeYuea%2FTTldEnDaq5izn%2FOZxOWEFm3669yGUnS9d50oCn2WppYZL%2FQpI8XrdpNJn6ex3fwFa1VpB9EEB%2Btfg3yu5qWJRa1g2zpfctV5F39dz9kDC4IWJm6yR63cTTIe6ZOIb%2BviRyJke4XQ8r2T6s96llOp%2F9udaxLgE4K9RK0w%2B8TtbC4J3wrN%2Bmq%2Bo6gIhGRw04D9dlb%2BGhlObY5LwH4ryr9l4GQ%3D&ddkey=https%3Ano-NO%2FElement14_Norway%2Fw%2Fc%2Fpassive-components%2Finductors%2Fpower-inductors%2Fsmd-power-inductors" V 1625 4275 50  0001 C CNN "Farnell"
+	1    1625 4275
+	0    -1   -1   0
+$EndComp
+Wire Wire Line
+	1725 4275 2175 4275
+Wire Wire Line
+	1525 4275 1375 4275
+Wire Wire Line
+	1375 4275 1375 4575
+Connection ~ 1375 4575
+Text Notes 1300 4050 0    50   ~ 0
+AVCC Lavpass filter
 $EndSCHEMATC

Commit message: Changelog for 30.07.2019
Parts:
- added C7: 100nF, Capacitor_SMD:C_0402_1005Metric, symbol Device:C
- C1: value 100n -> 100nF
- R1: Farnell (none) -> https://no.farnell.com/vishay/crcw0402100kfked/res-100k-1-0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
- U1: Farnell (none) -> https://no.farnell.com/microchip/atmega328pb-au/mcu-8bit-at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
Connections:
- net +5V: now also L1.1, U1.20 (AREF), C7.1; no longer L1.2, U1.18 (AVCC)
- net GND: now also C7.2
- new net: C6.2, L1.2, U1.18 (AVCC)
- no-connect marks 1 -> 0
Other:
- note added: "Close as possible to MCP-chip.\n Route on single layer with ground"
- note added: "Place as close as \npossible to pin 20"
- note removed: "Close as possible to MCP-chip"
- moved on the sheet: C1, C6, L1
