File: AR20_ECU/ECU_lambda_controller/ECU_lambda_circuit_diagram/lambda_controller_circuit/lambda_controller_circuit.sch (KiCad schematic (older format))
At the start: 3 parts

Commit message: .
Parts:
- added 6.8K: R, symbol Device:R
- added C3, C8, C? (x2): 33n, Capacitor_SMD:C_1206_3216Metric, symbol Device:C
- added C?: 1n, Capacitor_SMD:C_1206_3216Metric, symbol Device:C
- added R1: 10K, Capacitor_SMD:C_1206_3216Metric, symbol Device:R
- added R7: 31.6K, symbol Device:R
- added R?: 100K, symbol Device:R
- LDO1: renamed from LDO?; footprint (none) -> Package_TO_SOT_SMD:SOT-223
- MOSFET1: renamed from MOSFET?; footprint (none) -> Package_SO:SOIC-8-1EP_3.9x4.9mm_P1.27mm_EP2.29x3mm; symbol MCP_MOSFET:MCP14E10 -> lambda_controller_circuit-rescue:MCP14E10-MCP_MOSFET
- gave numbers to parts that had none: 1
Connections:
- net labels added: 5V, CJ124_UR, CJ125_DIAHG, CJ125_IA, CJ125_IP, CJ125_RESET, CJ125_RS, CJ125_UA, CJ125_UN, CJ125_UP, CJ125_US, GND
- wire segments 0 -> 31

Commit message: .
Parts:
- added 0.301K1: R9, Resistor_SMD:R_0603_1608Metric, symbol Device:R
- added C5, C6: 2.2uF, Capacitor_SMD:C_0603_1608Metric, symbol Device:C
- added R5: 100K, Resistor_SMD:R_0603_1608Metric, symbol Device:R
- added R6: 4.7K, Resistor_SMD:R_0603_1608Metric, symbol Device:R
- added R7: 470K, Resistor_SMD:R_0603_1608Metric, symbol Device:R
- added R8: 61.9, Resistor_SMD:R_0603_1608Metric, symbol Device:R
- 6.8K1: renamed from 6.8K; value R -> R2; footprint (none) -> Resistor_SMD:R_0603_1608Metric
- C1, C3, C4: renamed from C?; footprint Capacitor_SMD:C_1206_3216Metric -> Capacitor_SMD:C_0603_1608Metric
- C2: renamed from C8; footprint Capacitor_SMD:C_1206_3216Metric -> Capacitor_SMD:C_0603_1608Metric
- C7: renamed from C3; footprint Capacitor_SMD:C_1206_3216Metric -> Capacitor_SMD:C_0603_1608Metric
- R1: footprint Capacitor_SMD:C_1206_3216Metric -> Resistor_SMD:R_0603_1608Metric
- R3: renamed from R7; footprint (none) -> Resistor_SMD:R_0603_1608Metric
- R4: renamed from R?; footprint (none) -> Resistor_SMD:R_0603_1608Metric
Connections:
- net labels added: CJ125_SCK, CJ125_SI, CJ125_SO, CJ125_SS, CJ125_VM, LSU_IA, LSU_IP, LSU_UN, LSU_VM
- wire segments 31 -> 52
Other:
- moved on the sheet: C3
