File: AR20_ETC/AR20_ETBC/ETBC_schematics/AR20_ETBC_rev1/AR20_ETBC_rev1.sch (EAGLE design)
At the start: 29 parts, among them J1 1-776267-1, X3 22-23-2021

Commit message: .
Parts:
- removed U$1, U$2, U$5, U$6, U$7: 2PIN_TERMINAL_BLOCK, AR19_ETC:2PIN_TERMINAL_BLOCK
- removed X3: 22-23-2021, con-molex:22-23-2021
Connections:
- new net ECUTPS: J1.5
- new net N$16: J1.MH1
- new net N$22: J1.12
- new net N$24: J1.MH2
- new net SHUTD_IN: J1.8
- new net SHUTD_OUT: J1.9
- net 12V: now also J1.13; no longer U$2.P$2
- net 5V: now also J1.3; no longer U$6.P$2
- net CANH: now also J1.6; no longer U$1.P$2
- net CANL: now also J1.7; no longer U$1.P$1
- net GND: now also J1.14, J1.4; no longer U$2.P$1, U$6.P$1
- net OUT1: now also J1.10; no longer U$5.P$2
- net OUT2: now also J1.11; no longer U$5.P$1
- net PWM0: no longer X3-1.S
- net PWM1: no longer X3-2.S
- net TPS1: now also J1.1; no longer U$7.P$1
- net TPS2: now also J1.2; no longer U$7.P$2
Other:
- note removed: "1x2 Terminal Block Supply from LVMS"
- note removed: "3 pcs 1x2 Terminal Blocks to ETB (5mm Pitch)"
- note removed: "Test probes for PWM"
- moved on the sheet: J1
