File: AR20_ACM/ACM_pcb/01. KiCAD/ACM_Y2020V0.1/ACM_Y2020V0.1.kicad_pcb (KiCad board)
At the start: 2 copper layers, 18 x 22.5 mm, 30 parts, among them J1 TC2030-MCP-NL, P1 Conn_02x15_Odd_Even, Q1 Q_PMOS_DGS, U1 ATmega328PB-AU, U2 MCP25625-x-SS, U3 NCV890430MW50TXG, Y1 16.0Mhz

Commit message: Changelog for 04.08.2019
Parts:
- added C10: 10uF, Capacitor_SMD:C_0603_1608Metric, B.Cu at (134.3, 95.2)
- added C11: 10uF, Capacitor_SMD:C_0603_1608Metric, B.Cu at (137.4, 95.2)
- R1: value 10K -> 10K Ohm
- R6: value 10KOhm -> 10K Ohm
- R7: value 120Ohm -> 120 Ohm
- moved L2 1.69 mm to (135.8, 95.2), turned to 270 degrees
Other:
- board text added: "SN:"
- board text added: "[Optional]"

Commit message: Changelog for 06.10.2019
Parts:
- moved C9 0.75 mm to (138.4, 96.4)
- moved C7 0.39 mm to (142.3, 96.7)
Changed lines of the file:
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@@
   (page A4)
   (layers
-    (0 F.Cu signal hide)
-    (31 B.Cu signal)
+    (0 F.Cu signal)
+    (31 B.Cu signal hide)
     (32 B.Adhes user hide)
     (33 F.Adhes user hide)
-    (34 B.Paste user)
-    (35 F.Paste user hide)
-    (36 B.SilkS user)
-    (37 F.SilkS user hide)
-    (38 B.Mask user)
-    (39 F.Mask user hide)
+    (34 B.Paste user hide)
+    (35 F.Paste user)
+    (36 B.SilkS user hide)
+    (37 F.SilkS user)
+    (38 B.Mask user hide)
+    (39 F.Mask user)
     (40 Dwgs.User user hide)
     (41 Cmts.User user hide)
@@
     (44 Edge.Cuts user)
     (45 Margin user hide)
-    (46 B.CrtYd user)
-    (47 F.CrtYd user hide)
-    (48 B.Fab user)
-    (49 F.Fab user hide)
+    (46 B.CrtYd user hide)
+    (47 F.CrtYd user)
+    (48 B.Fab user hide)
+    (49 F.Fab user)
   )
   (setup
@@
   )
   (module Capacitor_SMD:C_0402_1005Metric (layer F.Cu)
-    (at 141.97 96.47 225)
+    (at 142.26824 96.72424 225)
     (descr "Capacitor SMD 0402 (1005 Metric), square (rectangular) end terminal, IPC_7351 nominal, (Body size source: http://www.tortai-tech.com/upload/download/2011102023233369053.pdf), generated with kicad-footprint-generator")
     (tags capacitor)
@@
     )
     (fp_text value 0.1uF (at 4.782945 3.090057 45) (layer F.Fab)
+      (effects (font (size 1 1) (thickness 0.15)))
+    )
+    (fp_line (start -0.5 0.25) (end -0.5 -0.25) (layer F.Fab) (width 0.1))
+    (fp_line (start -0.5 -0.25) (end 0.5 -0.25) (layer F.Fab) (width 0.1))
+    (fp_line (start 0.5 -0.25) (end 0.5 0.25) (layer F.Fab) (width 0.1))
+    (fp_line (start 0.5 0.25) (end -0.5 0.25) (layer F.Fab) (width 0.1))
+    (fp_line (start -0.93 0.47) (end -0.93 -0.47) (layer F.CrtYd) (width 0.05))
+    (fp_line (start -0.93 -0.47) (end 0.93 -0.47) (layer F.CrtYd) (width 0.05))
+    (fp_line (start 0.93 -0.47) (end 0.93 0.47) (layer F.CrtYd) (width 0.05))
+    (fp_line (start 0.93 0.47) (end -0.93 0.47) (layer F.CrtYd) (width 0.05))
+    (fp_text user %R (at -0.021553 -0.046697 45) (layer F.Fab)
+      (effects (font (size 0.25 0.25) (thickness 0.04)))
+    )
+    (pad 1 smd roundrect (at -0.485 0 225) (size 0.59 0.64) (layers F.Cu F.Paste F.Mask) (roundrect_rratio 0.25)
+      (net 51 "Net-(C7-Pad1)"))
+    (pad 2 smd roundrect (at 0.485 0 225) (size 0.59 0.64) (layers F.Cu F.Paste F.Mask) (roundrect_rratio 0.25)
+      (net 3 GND))
+    (model ${KISYS3DMOD}/Capacitor_SMD.3dshapes/C_0402_1005Metric.wrl
+      (at (xyz 0 0 0))
+      (scale (xyz 1 1 1))
+      (rotate (xyz 0 0 0))
+    )
+  )
+  (module Capacitor_SMD:C_0402_1005Metric (layer F.Cu)
+    (at 136.78 89.88 225)
+    (descr "Capacitor SMD 0402 (1005 Metric), square (rectangular) end terminal, IPC_7351 nominal, (Body size source: http://www.tortai-tech.com/upload/download/2011102023233369053.pdf), generated with kicad-footprint-generator")
+    (tags capacitor)
+    (attr smd)
+    (fp_text reference C8 (at 1.880904 -0.311127 225) (layer F.SilkS)
+      (effects (font (size 1 1) (thickness 0.15)))
+    )
+    (fp_text value 0.1uF (at 0 1.17 45) (layer F.Fab) hide
       (effects (font (size 1 1) (thickness 0.15)))
     )
@@
   )
   (module Capacitor_SMD:C_0402_1005Metric (layer F.Cu)
-    (at 136.78 89.88 225)
+    (at 138.36172 96.43214 45)
     (descr "Capacitor SMD 0402 (1005 Metric), square (rectangular) end terminal, IPC_7351 nominal, (Body size source: http://www.tortai-tech.com/upload/download/2011102023233369053.pdf), generated with kicad-footprint-generator")
     (tags capacitor)
     (attr smd)
-    (fp_text reference C8 (at 1.880904 -0.311127 225) (layer F.SilkS)
-      (effects (font (size 1 1) (thickness 0.15)))
-    )
-    (fp_text value 0.1uF (at 0 1.17 45) (layer F.Fab) hide
+    (fp_text reference C9 (at -1.895046 -0.212132) (layer F.SilkS)
+      (effects (font (size 1 1) (thickness 0.15)))
+    )
+    (fp_text value 0.1uF (at -5.041671 3.599174 45) (layer F.Fab)
       (effects (font (size 1 1) (thickness 0.15)))
     )
@@
     (fp_line (start 0.93 -0.47) (end 0.93 0.47) (layer F.CrtYd) (width 0.05))
     (fp_line (start 0.93 0.47) (end -0.93 0.47) (layer F.CrtYd) (width 0.05))
-    (fp_text user %R (at 0 0 45) (layer F.Fab)
+    (fp_text user %R (at -0.003592 -0.050289 45) (layer F.Fab)
       (effects (font (size 0.25 0.25) (thickness 0.04)))
     )
-    (pad 1 smd roundrect (at -0.485 0 225) (size 0.59 0.64) (layers F.Cu F.Paste F.Mask) (roundrect_rratio 0.25)
-      (net 51 "Net-(C7-Pad1)"))
-    (pad 2 smd roundrect (at 0.485 0 225) (size 0.59 0.64) (layers F.Cu F.Paste F.Mask) (roundrect_rratio 0.25)
-      (net 3 GND))
-    (model ${KISYS3DMOD}/Capacitor_SMD.3dshapes/C_0402_1005Metric.wrl
-      (at (xyz 0 0 0))
-      (scale (xyz 1 1 1))
-      (rotate (xyz 0 0 0))
-    )
-  )
-  (module Capacitor_SMD:C_0402_1005Metric (layer F.Cu)
-    (at 138.92 95.93 45)
-    (descr "Capacitor SMD 0402 (1005 Metric), square (rectangular) end terminal, IPC_7351 nominal, (Body size source: http://www.tortai-tech.com/upload/download/2011102023233369053.pdf), generated with kicad-footprint-generator")
-    (tags capacitor)
-    (attr smd)
-    (fp_text reference C9 (at -1.895046 -0.212132) (layer F.SilkS)
-      (effects (font (size 1 1) (thickness 0.15)))
-    )
-    (fp_text value 0.1uF (at -5.041671 3.599174 45) (layer F.Fab)
-      (effects (font (size 1 1) (thickness 0.15)))
-    )
-    (fp_line (start -0.5 0.25) (end -0.5 -0.25) (layer F.Fab) (width 0.1))
-    (fp_line (start -0.5 -0.25) (end 0.5 -0.25) (layer F.Fab) (width 0.1))
-    (fp_line (start 0.5 -0.25) (end 0.5 0.25) (layer F.Fab) (width 0.1))
-    (fp_line (start 0.5 0.25) (end -0.5 0.25) (layer F.Fab) (width 0.1))
-    (fp_line (start -0.93 0.47) (end -0.93 -0.47) (layer F.CrtYd) (width 0.05))
-    (fp_line (start -0.93 -0.47) (end 0.93 -0.47) (layer F.CrtYd) (width 0.05))
-    (fp_line (start 0.93 -0.47) (end 0.93 0.47) (layer F.CrtYd) (width 0.05))
-    (fp_line (start 0.93 0.47) (end -0.93 0.47) (layer F.CrtYd) (width 0.05))
-    (fp_text user %R (at -0.021213 -0.035355 45) (layer F.Fab)
-      (effects (font (size 0.25 0.25) (thickness 0.04)))
-    )

Commit message: Changelog for 06.10.2019
Parts:
- U1: value ATmega328PB-AU -> ATmega328P-AU
- moved C1 0.92 mm to (137.3, 77.4)
Connections:
- U1 pad 1: /U-Pin20 -> Net-(U1-Pad1)
- U1 pad 19: /U-Pin11 -> Net-(U1-Pad19)
- U1 pad 2: /U-Pin22 -> Net-(U1-Pad2)
- U1 pad 22: /U-Pin9 -> Net-(U1-Pad22)
- U1 pad 23: /U-Pin7 -> Net-(U1-Pad23)
- U1 pad 24: /U-Pin5 -> Net-(U1-Pad24)
- U1 pad 3: /U-Pin24 -> GND
- U1 pad 6: /U-Pin30 -> +5V
