File: AR20_ACM/ACM_pcb/01. KiCAD/ACM_Y2020V0.1/ACM_Y2020V0.1.sch (KiCad schematic (older format))
At the start: 26 parts, among them J1 TC2030-MCP-NL, J2 Conn_02x15_Odd_Even, Q1 Q_PMOS_DGS, U1 ATmega328PB-AU, U2 MCP25625-x-SS, U3 SPX3819M5-L-5-0, Y1 16.0Mhz

Commit message: Changelog for 03.08.2019
Parts:
- removed U3: SPX3819M5-L-5-0, Package_TO_SOT_SMD:SOT-23-5, symbol Regulator_Linear:SPX3819M5-L-5-0
- added C4, C5: 0.1uF, Capacitor_SMD:C_0402_1005Metric, symbol Device:C
- added H1: M2 Mouting hole, MountingHole:MountingHole_2.2mm_M2, symbol Mechanical:MountingHole
- added L2: 2.2 µH, Inductor_SMD:L_0603_1608Metric, symbol Device:L_Small
- added U3: NCV890430MW50TXG, NCV890430MW50TXG:SON65P300X300X100-9N, symbol NCV890430MW50TXG:NCV890430MW50TXG
- C1: value 100nF -> 0.1uF
- C2: renamed from C?; value 100nF -> 0.1uF
- C3: renamed from C6; value 100nF -> 0.1uF
- P1: renamed from J2; footprint Connector_PinSocket_0.8mm:PinSocket_2x15_P0.08mm_Vertical_SMD -> SMLP36RGB2W3R:ILWX10SBVFBE
- renumbered C5 to C6, C2 to C7, C3 to C8, C4 to C9, R7 to R2, R4 to R3, R5 to R4, R6 to R5, R3 to R6, R2 to R7
Connections:
- net labels added: +12V_Safe
- wire segments 98 -> 115
Other:
- note added: "Mechanical"
- moved on the sheet: D1, D2, F1, Q1, R2

Commit message: Changelog for 04.08.2019
Parts:
- added C10, C11: 10uF, Capacitor_SMD:C_0603_1608Metric, symbol Device:C
- R1: value 10K -> 10K Ohm
- R6: value 10KOhm -> 10K Ohm
- R7: value 120Ohm -> 120 Ohm
Connections:
- net +12V_Safe: now also C10.1
- net +5V: now also C11.1
- net GND: now also C10.2, C11.2
Changed lines of the file:
@@
 F 3 "http://ww1.microchip.com/downloads/en/DeviceDoc/TC2030-MCP-NL_PCB_Footprint_RevD.pdf" H 2925 1400 50  0001 L CNN
 F 4 "TC2030-MCP-NL PCB Footprint (no legs)" H 2925 1300 50  0001 L CNN "Description"
-F 5 "" H 2925 1200 50  0001 L CNN "Height"
-F 6 "Microchip" H 2925 1100 50  0001 L CNN "Manufacturer_Name"
-F 7 "TC2030-MCP-NL" H 2925 1000 50  0001 L CNN "Manufacturer_Part_Number"
-F 8 "579-TC2030-MCP-NL" H 2925 900 50  0001 L CNN "Mouser Part Number"
-F 9 "https://www.mouser.com/Search/Refine.aspx?Keyword=579-TC2030-MCP-NL" H 2925 800 50  0001 L CNN "Mouser Price/Stock"
-F 10 "8252561" H 2925 700 50  0001 L CNN "RS Part Number"
-F 11 "http://uk.rs-online.com/web/p/products/8252561" H 2925 600 50  0001 L CNN "RS Price/Stock"
+F 5 "Microchip" H 2925 1100 50  0001 L CNN "Manufacturer_Name"
+F 6 "TC2030-MCP-NL" H 2925 1000 50  0001 L CNN "Manufacturer_Part_Number"
+F 7 "579-TC2030-MCP-NL" H 2925 900 50  0001 L CNN "Mouser Part Number"
+F 8 "https://www.mouser.com/Search/Refine.aspx?Keyword=579-TC2030-MCP-NL" H 2925 800 50  0001 L CNN "Mouser Price/Stock"
+F 9 "8252561" H 2925 700 50  0001 L CNN "RS Part Number"
+F 10 "http://uk.rs-online.com/web/p/products/8252561" H 2925 600 50  0001 L CNN "RS Price/Stock"
 	1    1075 1400
 	1    0    0    -1
@@
 P 3275 5850
 F 0 "R1" H 3345 5896 50  0000 L CNN
-F 1 "10K" H 3345 5805 50  0000 L CNN
+F 1 "10K Ohm" H 3345 5805 50  0000 L CNN
 F 2 "Resistor_SMD:R_0402_1005Metric" V 3205 5850 50  0001 C CNN
 F 3 "http://www.farnell.com/datasheets/2310790.pdf?_ga=2.87708376.1939358490.1564414725-1415930916.1560114588&_gac=1.257050489.1564075292.CjwKCAjwpuXpBRAAEiwAyRRPgXwHZ1wF4xXBoNI_FJEvoVORJn7NbJB9jjbidsg8_qDnlLi_44u6wRoCV2MQAvD_BwE" H 3275 5850 50  0001 C CNN
@@
 P 10325 4050
 F 0 "R7" H 10395 4096 50  0000 L CNN
-F 1 "120Ohm" H 10395 4005 50  0000 L CNN
+F 1 "120 Ohm" H 10395 4005 50  0000 L CNN
 F 2 "Resistor_SMD:R_0603_1608Metric" V 10255 4050 50  0001 C CNN
 F 3 "~" H 10325 4050 50  0001 C CNN
@@
 P 8475 4700
 F 0 "R6" V 8268 4700 50  0000 C CNN
-F 1 "10KOhm" V 8359 4700 50  0000 C CNN
+F 1 "10K Ohm" V 8359 4700 50  0000 C CNN
 F 2 "Resistor_SMD:R_0402_1005Metric" V 8405 4700 50  0001 C CNN
 F 3 "~" H 8475 4700 50  0001 C CNN
@@
 F 3 "http://www.rohm.com/web/global/datasheet/SMLP36RGB2W(R)" H 9925 1450 50  0001 L CNN
 F 4 "LED,RGB,35/110/35mcd,top-looking,1510 ROHM SMLP36RGB2W3R, SML-P36 Series 3 RGB LED, 475 (Blue) nm, 535 (Green) nm, 629 (Red) nm 6-Pin Milky White" H 9925 1350 50  0001 L CNN "Description"
-F 5 "" H 9925 1250 50  0001 L CNN "Height"
-F 6 "ROHM Semiconductor" H 9925 1150 50  0001 L CNN "Manufacturer_Name"
-F 7 "SMLP36RGB2W3R" H 9925 1050 50  0001 L CNN "Manufacturer_Part_Number"
-F 8 "755-SMLP36RGB2W3R" H 9925 950 50  0001 L CNN "Mouser Part Number"
-F 9 "https://www.mouser.com/Search/Refine.aspx?Keyword=755-SMLP36RGB2W3R" H 9925 850 50  0001 L CNN "Mouser Price/Stock"
-F 10 "1246884" H 9925 750 50  0001 L CNN "RS Part Number"
-F 11 "https://uk.rs-online.com/web/p/products/1246884" H 9925 650 50  0001 L CNN "RS Price/Stock"
+F 5 "ROHM Semiconductor" H 9925 1150 50  0001 L CNN "Manufacturer_Name"
+F 6 "SMLP36RGB2W3R" H 9925 1050 50  0001 L CNN "Manufacturer_Part_Number"
+F 7 "755-SMLP36RGB2W3R" H 9925 950 50  0001 L CNN "Mouser Part Number"
+F 8 "https://www.mouser.com/Search/Refine.aspx?Keyword=755-SMLP36RGB2W3R" H 9925 850 50  0001 L CNN "Mouser Price/Stock"
+F 9 "1246884" H 9925 750 50  0001 L CNN "RS Part Number"
+F 10 "https://uk.rs-online.com/web/p/products/1246884" H 9925 650 50  0001 L CNN "RS Price/Stock"
 	1    8575 1450
 	1    0    0    -1
@@
 U 1 1 5D471BBC
 P 7225 5950
-F 0 "C5" H 7340 5996 50  0000 L CNN
-F 1 "0.1uF" H 7340 5905 50  0000 L CNN
+F 0 "C5" H 7025 6025 50  0000 L CNN
+F 1 "0.1uF" H 6925 5925 50  0000 L CNN
 F 2 "Capacitor_SMD:C_0402_1005Metric" H 7263 5800 50  0001 C CNN
 F 3 "~" H 7225 5950 50  0001 C CNN
@@
 Text GLabel 6125 4950 2    50   Input ~ 0
 +12V_Safe
-Text GLabel 5025 5800 0    50   Input ~ 0
+Text GLabel 4625 5725 1    50   Input ~ 0
 +12V_Safe
-Wire Wire Line
-	5025 5800 5175 5800
 Wire Wire Line
 	5175 6025 5175 5800
@@
 Wire Wire Line
 	7075 5800 7225 5800
-Connection ~ 7475 5800
-Wire Wire Line
-	7475 5800 7575 5800
+Connection ~ 7600 5800
+Wire Wire Line
+	7600 5800 7700 5800
 Wire Wire Line
 	6725 6100 6825 6100
@@
 	6825 6100 6825 6075
 Wire Wire Line
-	6825 6075 7475 6075
-Wire Wire Line
-	7475 6075 7475 5800
+	7600 6075 7600 5800
 Connection ~ 7225 5800
 Wire Wire Line
-	7225 5800 7475 5800
-Wire Wire Line
-	7575 5800 7575 5700
+	7700 5800 7700 5700
 $Comp
 L power:+5V #PWR022
 U 1 1 5D4DE85A
-P 7575 5700
-F 0 "#PWR022" H 7575 5550 50  0001 C CNN
-F 1 "+5V" H 7590 5873 50  0000 C CNN
-F 2 "" H 7575 5700 50  0001 C CNN
-F 3 "" H 7575 5700 50  0001 C CNN
-	1    7575 5700
-	1    0    0    -1
-$EndComp
+P 7700 5700
+F 0 "#PWR022" H 7700 5550 50  0001 C CNN
+F 1 "+5V" H 7715 5873 50  0000 C CNN
+F 2 "" H 7700 5700 50  0001 C CNN
+F 3 "" H 7700 5700 50  0001 C CNN
+	1    7700 5700
+	1    0    0    -1
+$EndComp
+$Comp
+L Device:C C11
+U 1 1 5D4736E4
+P 7450 5950
+F 0 "C11" H 7565 5996 50  0000 L CNN
+F 1 "10uF" H 7565 5905 50  0000 L CNN
+F 2 "Capacitor_SMD:C_0603_1608Metric" H 7488 5800 50  0001 C CNN
+F 3 "~" H 7450 5950 50  0001 C CNN
+	1    7450 5950
+	1    0    0    -1
+$EndComp
+Wire Wire Line
+	7225 5800 7450 5800
+Wire Wire Line
+	7450 5800 7600 5800
+Connection ~ 7450 5800
+$Comp
+L power:GND #PWR0101
+U 1 1 5D486DC3
+P 7450 6100
+F 0 "#PWR0101" H 7450 5850 50  0001 C CNN
+F 1 "GND" H 7455 5927 50  0000 C CNN
+F 2 "" H 7450 6100 50  0001 C CNN
+F 3 "" H 7450 6100 50  0001 C CNN
+	1    7450 6100
+	1    0    0    -1
+$EndComp
+$Comp
+L Device:C C10
+U 1 1 5D487807
+P 4750 6200
+F 0 "C10" H 4865 6246 50  0000 L CNN
+F 1 "10uF" H 4865 6155 50  0000 L CNN
+F 2 "Capacitor_SMD:C_0603_1608Metric" H 4788 6050 50  0001 C CNN
+F 3 "~" H 4750 6200 50  0001 C CNN
+	1    4750 6200
+	-1   0    0    -1
+$EndComp
+Wire Wire Line
+	4625 5800 4625 5725
+Wire Wire Line
+	4625 5800 4750 5800
+Wire Wire Line
+	4750 6050 4750 5800
+Connection ~ 4750 5800
+Wire Wire Line
+	4750 5800 5175 5800
+$Comp
+L power:GND #PWR0102
+U 1 1 5D49183D
+P 4750 6350
+F 0 "#PWR0102" H 4750 6100 50  0001 C CNN
+F 1 "GND" H 4755 6177 50  0000 C CNN
+F 2 "" H 4750 6350 50  0001 C CNN
+F 3 "" H 4750 6350 50  0001 C CNN
+	1    4750 6350
+	1    0    0    -1
+$EndComp
+Wire Wire Line
+	6825 6075 7600 6075
 $EndSCHEMATC

Commit message: Changelog for 06.10.2019
Parts:
- J1: symbol TC2030-MCP-NL:TC2030-MCP-NL -> ACM_Y2020V0.1-rescue:TC2030-MCP-NL-TC2030-MCP-NL
- LED1: symbol SMLP36RGB2W3R:SMLP36RGB2W3R -> ACM_Y2020V0.1-rescue:SMLP36RGB2W3R-SMLP36RGB2W3R
- U3: symbol NCV890430MW50TXG:NCV890430MW50TXG -> ACM_Y2020V0.1-rescue:NCV890430MW50TXG-NCV890430MW50TXG
Changed lines of the file:
@@
 $EndDescr
 $Comp
-L TC2030-MCP-NL:TC2030-MCP-NL J1
+L ACM_Y2020V0.1-rescue:TC2030-MCP-NL-TC2030-MCP-NL J1
 U 1 1 5D389624
 P 1075 1400
@@
 $EndComp
 $Comp
-L SMLP36RGB2W3R:SMLP36RGB2W3R LED1
+L ACM_Y2020V0.1-rescue:SMLP36RGB2W3R-SMLP36RGB2W3R LED1
 U 1 1 5D41B8EC
 P 8575 1450
@@
 	1750 2525 575  2525
 $Comp
-L NCV890430MW50TXG:NCV890430MW50TXG U3
+L ACM_Y2020V0.1-rescue:NCV890430MW50TXG-NCV890430MW50TXG U3
 U 1 1 5D46D022
 P 5525 5800

Commit message: Changelog for 06.10.2019
Parts:
- removed U1: ATmega328PB-AU, Package_QFP:TQFP-32_7x7mm_P0.8mm, symbol MCU_Microchip_ATmega:ATmega328PB-AU
- added U?: ATmega328P-AU, Package_QFP:TQFP-32_7x7mm_P0.8mm, symbol MCU_Microchip_ATmega:ATmega328P-AU
Connections:
- net +5V: now also U?.20 (AREF), U?.4 (VCC), U?.6 (VCC)
- net GND: now also U?.21 (GND), U?.3 (GND), U?.5 (GND)
- net Reset: now also U?.29 (~RESET~/PC6)
- net at C3.2, L1.2: now also U?.18 (AVCC)
- net at Y1.3: now also U?.7 (XTAL1/PB6)
- net at Y1.1: now also U?.8 (XTAL2/PB7)
Other:
- moved on the sheet: C2
Changed lines of the file:
@@
 	1    0    0    -1
 $EndComp
-Wire Wire Line
-	2175 4125 2175 4275
 $Comp
 L Device:C C1
@@
 	1    0    0    -1
 $EndComp
-Wire Wire Line
-	2775 6075 3275 6075
 $Comp
 L power:+5V #PWR09
@@
 	1    0    0    -1
 $EndComp
-Text HLabel 2775 6975 2    50   Input ~ 0
+Text HLabel 2850 6975 2    50   Input ~ 0
 CAN_CS
 Text HLabel 8875 4500 0    50   Input ~ 0
@@
 	1    0    0    -1
 $EndComp
-Text HLabel 2775 6475 2    50   Input ~ 0
+Text HLabel 2850 6475 2    50   Input ~ 0
 CAN_INT
 Text HLabel 8875 5600 0    50   Input ~ 0
@@
 Wire Wire Line
 	10175 1450 10175 1375
-Text HLabel 2775 6775 2    50   Input ~ 0
+Text HLabel 2850 6775 2    50   Input ~ 0
 GREEN_LED
 $Comp
@@
 Wire Wire Line
 	6025 1875 6425 1875
-Text HLabel 1575 6275 0    50   Input ~ 0
+Text HLabel 1400 6300 0    50   Input ~ 0
 U-Pin24
-Text HLabel 1575 6375 0    50   Input ~ 0
+Text HLabel 1400 6400 0    50   Input ~ 0
 U-Pin30
-Text HLabel 1575 6475 0    50   Input ~ 0
+Text HLabel 1400 6500 0    50   Input ~ 0
 U-Pin11
-Text HLabel 1575 6575 0    50   Input ~ 0
+Text HLabel 1400 6600 0    50   Input ~ 0
 U-Pin9
-Text HLabel 2775 6675 2    50   Input ~ 0
+Text HLabel 2850 6675 2    50   Input ~ 0
 U-Pin22
-Text HLabel 2775 6575 2    50   Input ~ 0
+Text HLabel 2850 6575 2    50   Input ~ 0
 U-Pin20
-Text HLabel 2775 6375 2    50   Input ~ 0
+Text HLabel 2850 6375 2    50   Input ~ 0
 U-Pin14
-Text HLabel 2775 6275 2    50   Input ~ 0
+Text HLabel 2850 6275 2    50   Input ~ 0
 U-Pin12
-Connection ~ 3275 6075
 Wire Wire Line
 	3275 6075 3275 6000
-Text HLabel 2775 5975 2    50   Input ~ 0
+Text HLabel 2825 5975 2    50   Input ~ 0
 U-Pin8
-Text HLabel 2775 5875 2    50   Input ~ 0
+Text HLabel 2825 5875 2    50   Input ~ 0
 U-Pin6
-Text HLabel 2775 5775 2    50   Input ~ 0
+Text HLabel 2825 5775 2    50   Input ~ 0
 U-Pin4
-Text HLabel 2775 5675 2    50   Input ~ 0
+Text HLabel 2825 5675 2    50   Input ~ 0
 U-Pin2
-Text HLabel 2775 5575 2    50   Input ~ 0
-U-Pin5
-Text HLabel 2775 5475 2    50   Input ~ 0
+Text HLabel 2825 5475 2    50   Input ~ 0
 U-Pin7
 Text HLabel 10775 3900 2    50   Input ~ 0
@@
 Wire Wire Line
 	3500 5275 2775 5275
-Text HLabel 2775 6875 2    50   Input ~ 0
+Text HLabel 2850 6875 2    50   Input ~ 0
 U-Pin23
 Text HLabel 5900 1575 2    50   Input ~ 0
@@
 AVCC Lavpass filter
 Wire Wire Line
-	2275 4275 2275 4250
-Wire Wire Line
-	2275 4250 2700 4250
-Wire Wire Line
-	2700 4250 2700 4125
-Wire Wire Line
 	2850 4125 2700 4125
 Connection ~ 2700 4125
@@
 	2400 4125 2175 4125
 Connection ~ 2175 4125
-Wire Wire Line
-	1550 4125 2175 4125
-Text Notes 1500 4575 2    50   ~ 0
+Text Notes 1150 4600 2    50   ~ 0
 Place as close as \npossible to pin 20
-Connection ~ 1550 4575
 $Comp
 L power:GND #PWR03
 U 1 1 5D434DF4
-P 1550 4875
-F 0 "#PWR03" H 1550 4625 50  0001 C CNN
-F 1 "GND" H 1555 4702 50  0000 C CNN
-F 2 "" H 1550 4875 50  0001 C CNN
-F 3 "" H 1550 4875 50  0001 C CNN
-	1    1550 4875
+P 1300 4925
+F 0 "#PWR03" H 1300 4675 50  0001 C CNN
+F 1 "GND" H 1305 4752 50  0000 C CNN
+F 2 "" H 1300 4925 50  0001 C CNN
+F 3 "" H 1300 4925 50  0001 C CNN
+	1    1300 4925
 	1    0    0    -1
 $EndComp
@@
 L Device:C C2
 U 1 1 5D434DE8
-P 1550 4725
-F 0 "C2" H 1350 4825 50  0000 L CNN
-F 1 "0.1uF" H 1250 4725 50  0000 L CNN
-F 2 "Capacitor_SMD:C_0402_1005Metric" H 1588 4575 50  0001 C CNN
-F 3 "~" H 1550 4725 50  0001 C CNN
-	1    1550 4725
-	1    0    0    -1
-$EndComp
-Wire Wire Line
-	1550 4575 1550 4125
-Wire Wire Line
-	1575 4575 1550 4575
-Wire Wire Line
-	2775 4975 2850 4975
-Wire Wire Line
-	2775 4875 2850 4875
-Wire Wire Line
-	2775 4775 2875 4775
-Wire Wire Line
-	2775 4675 2850 4675
+P 1300 4775
+F 0 "C2" H 1100 4875 50  0000 L CNN
+F 1 "0.1uF" H 1000 4775 50  0000 L CNN
+F 2 "Capacitor_SMD:C_0402_1005Metric" H 1338 4625 50  0001 C CNN
+F 3 "~" H 1300 4775 50  0001 C CNN
+	1    1300 4775
+	1    0    0    -1
+$EndComp
 Wire Wire Line
 	3500 5175 3500 5150
@@
 Wire Wire Line
 	3500 5150 3600 5150
-Text Notes 3200 4675 0    50   ~ 0
+Text Notes 3150 4600 0    50   ~ 0
 Close as possible to MCP-chip.\n    Route on single layer with ground
-Text HLabel 2775 4575 2    50   Input ~ 0
+Text HLabel 2850 4575 2    50   Input ~ 0
 CLK_MCP
-$Comp
-L MCU_Microchip_ATmega:ATmega328PB-AU U1
-U 1 1 5D38D7A6
-P 2175 5775
-F 0 "U1" H 2375 4325 50  0000 L CNN
-F 1 "ATmega328PB-AU" H 2625 4250 50  0000 L CNN
-F 2 "Package_QFP:TQFP-32_7x7mm_P0.8mm" H 2175 5775 50  0001 C CIN
-F 3 "http://ww1.microchip.com/downloads/en/DeviceDoc/40001906C.pdf" H 2175 5775 50  0001 C CNN
-F 4 "https://no.farnell.com/microchip/atmega328pb-au/mcu-8bit-atmega-20mhz-tqfp-32/dp/2523203?st=ATMEGA328p" H 2175 5775 50  0001 C CNN "Farnell"
-	1    2175 5775
-	1    0    0    -1
-$EndComp
 $Comp
 L Device:Resonator_Small Y1
@@
 Text HLabel 2850 4975 2    50   Input ~ 0
 MISO
-Text HLabel 2775 5075 2    50   Input ~ 0
+Text HLabel 2825 5075 2    50   Input ~ 0
 SCK
 $Comp
@@
 Wire Wire Line
 	6825 6075 7600 6075
+$Comp
+L MCU_Microchip_ATmega:ATmega328P-AU U?
+U 1 1 5D9A1492
+P 2175 5775
+F 0 "U?" H 2575 4300 50  0000 C CNN
+F 1 "ATmega328P-AU" H 2575 4200 50  0000 C CNN
+F 2 "Package_QFP:TQFP-32_7x7mm_P0.8mm" H 2175 5775 50  0001 C CIN
+F 3 "http://ww1.microchip.com/downloads/en/DeviceDoc/ATmega328_P%20AVR%20MCU%20with%20picoPower%20Technology%20Data%20Sheet%2040001984A.pdf" H 2175 5775 50  0001 C CNN
+	1    2175 5775
+	1    0    0    -1
+$EndComp
+Text HLabel 2825 5575 2    50   Input ~ 0
+U-Pin5
+Wire Wire Line
+	2175 4100 2175 4125
+Wire Wire Line
+	2175 4125 2175 4275
+Wire Wire Line
+	2275 4275 2700 4275
+Wire Wire Line
+	2700 4125 2700 4275
+Wire Wire Line
+	2775 6075 3275 6075
+Connection ~ 3275 6075
+Wire Wire Line
+	1575 4575 1300 4575
+Wire Wire Line
+	1300 4575 1300 4625
+Wire Wire Line
+	1300 4575 1300 4125
+Wire Wire Line
+	1300 4125 2175 4125
+Connection ~ 1300 4575
 $EndSCHEMATC

Commit message: Changelog for 06.10.2019
Parts:
- gave numbers to parts that had none: 1
Connections:
- net BLUE_LED: now also U1.14 (PB2)
- net CAN_CS: now also U1.11 (PD7)
- net CAN_INT: now also U1.32 (PD2)
- net CLK_MCP: now also U1.12 (PB0)
- net GREEN_LED: now also U1.9 (PD5)
- net MISO: now also U1.16 (PB4)
- net MOSI: now also U1.15 (PB3)
- net RED_LED: now also U1.13 (PB1)
- net SCK: now also U1.17 (PB5)
- net U-Pin12: now also U1.30 (PD0)
- net U-Pin14: now also U1.31 (PD1)
- net U-Pin2: now also U1.25 (PC2)
- net U-Pin20: now also U1.1 (PD3)
- net U-Pin22: now also U1.2 (PD4)
- net U-Pin23: now also U1.10 (PD6)
- net U-Pin4: now also U1.26 (PC3)
- net U-Pin5: now also U1.24 (PC1)
- net U-Pin6: now also U1.27 (PC4)
- net U-Pin7: now also U1.23 (PC0)
- net U-Pin8: now also U1.28 (PC5)
Changed lines of the file:
@@
 	1    0    0    -1
 $EndComp
-Text HLabel 2850 6975 2    50   Input ~ 0
+Text HLabel 2775 6975 2    50   Input ~ 0
 CAN_CS
 Text HLabel 8875 4500 0    50   Input ~ 0
@@
 	1    0    0    -1
 $EndComp
-Text HLabel 2850 6475 2    50   Input ~ 0
+Text HLabel 2775 6475 2    50   Input ~ 0
 CAN_INT
 Text HLabel 8875 5600 0    50   Input ~ 0
@@
 Wire Wire Line
 	10175 1450 10175 1375
-Text HLabel 2850 6775 2    50   Input ~ 0
+Text HLabel 2775 6775 2    50   Input ~ 0
 GREEN_LED
 $Comp
@@
 Text HLabel 1400 6600 0    50   Input ~ 0
 U-Pin9
-Text HLabel 2850 6675 2    50   Input ~ 0
+Text HLabel 2775 6675 2    50   Input ~ 0
 U-Pin22
-Text HLabel 2850 6575 2    50   Input ~ 0
+Text HLabel 2775 6575 2    50   Input ~ 0
 U-Pin20
-Text HLabel 2850 6375 2    50   Input ~ 0
+Text HLabel 2775 6375 2    50   Input ~ 0
 U-Pin14
-Text HLabel 2850 6275 2    50   Input ~ 0
+Text HLabel 2775 6275 2    50   Input ~ 0
 U-Pin12
 Wire Wire Line
 	3275 6075 3275 6000
-Text HLabel 2825 5975 2    50   Input ~ 0
+Text HLabel 2775 5975 2    50   Input ~ 0
 U-Pin8
-Text HLabel 2825 5875 2    50   Input ~ 0
+Text HLabel 2775 5875 2    50   Input ~ 0
 U-Pin6
-Text HLabel 2825 5775 2    50   Input ~ 0
+Text HLabel 2775 5775 2    50   Input ~ 0
 U-Pin4
-Text HLabel 2825 5675 2    50   Input ~ 0
+Text HLabel 2775 5675 2    50   Input ~ 0
 U-Pin2
-Text HLabel 2825 5475 2    50   Input ~ 0
+Text HLabel 2775 5475 2    50   Input ~ 0
 U-Pin7
 Text HLabel 10775 3900 2    50   Input ~ 0
@@
 Wire Wire Line
 	3500 5275 2775 5275
-Text HLabel 2850 6875 2    50   Input ~ 0
+Text HLabel 2775 6875 2    50   Input ~ 0
 U-Pin23
 Text HLabel 5900 1575 2    50   Input ~ 0
@@
 Wire Wire Line
 	3500 5175 3500 5150
-Text HLabel 2875 4775 2    50   Input ~ 0
+Text HLabel 2775 4775 2    50   Input ~ 0
 BLUE_LED
-Text HLabel 2850 4675 2    50   Input ~ 0
+Text HLabel 2775 4675 2    50   Input ~ 0
 RED_LED
 Wire Notes Line
@@
 Text Notes 3150 4600 0    50   ~ 0
 Close as possible to MCP-chip.\n    Route on single layer with ground
-Text HLabel 2850 4575 2    50   Input ~ 0
+Text HLabel 2775 4575 2    50   Input ~ 0
 CLK_MCP
 $Comp
@@
 	0    -1   -1   0
 $EndComp
-Text HLabel 2850 4875 2    50   Input ~ 0
+Text HLabel 2775 4875 2    50   Input ~ 0
 MOSI
-Text HLabel 2850 4975 2    50   Input ~ 0
+Text HLabel 2775 4975 2    50   Input ~ 0
 MISO
-Text HLabel 2825 5075 2    50   Input ~ 0
+Text HLabel 2775 5075 2    50   Input ~ 0
 SCK
 $Comp
@@
 	6825 6075 7600 6075
 $Comp
-L MCU_Microchip_ATmega:ATmega328P-AU U?
+L MCU_Microchip_ATmega:ATmega328P-AU U1
 U 1 1 5D9A1492
 P 2175 5775
-F 0 "U?" H 2575 4300 50  0000 C CNN
+F 0 "U1" H 2575 4300 50  0000 C CNN
 F 1 "ATmega328P-AU" H 2575 4200 50  0000 C CNN
 F 2 "Package_QFP:TQFP-32_7x7mm_P0.8mm" H 2175 5775 50  0001 C CIN
@@
 	1    0    0    -1
 $EndComp
-Text HLabel 2825 5575 2    50   Input ~ 0
+Text HLabel 2775 5575 2    50   Input ~ 0
 U-Pin5
 Wire Wire Line
