File: AR20_CPU/Voltage_divider_PCB/VoltageDivider5Vto 3.1V/Teensy4_header_breakout/VoltageDivider/VoltageDivider.kicad_pcb (KiCad board)
At the start: 2 copper layers, 24.1 x 21.6 mm, 18 parts

Commit message: PCB VD finished
Parts:
- added TP1: TestPoint, TestPoint:TestPoint_THTPad_D1.0mm_Drill0.5mm, F.Cu at (145.8, 77.5)
- added TP2: TestPoint, TestPoint:TestPoint_THTPad_D1.0mm_Drill0.5mm, F.Cu at (145.8, 87.4)
- added TP3: TestPoint, TestPoint:TestPoint_THTPad_D1.0mm_Drill0.5mm, F.Cu at (165.1, 77.5)
- added TP4: TestPoint, TestPoint:TestPoint_THTPad_D1.0mm_Drill0.5mm, F.Cu at (165.0, 87.2)
- added TP5: TestPoint, TestPoint:TestPoint_THTPad_D1.0mm_Drill0.5mm, F.Cu at (153.8, 91.1)
- added TP6: TestPoint, TestPoint:TestPoint_THTPad_D1.0mm_Drill0.5mm, F.Cu at (151.8, 91.1)
- added TP7: TestPoint, TestPoint:TestPoint_THTPad_D1.0mm_Drill0.5mm, F.Cu at (157.9, 91.1)
- added TP8: TestPoint, TestPoint:TestPoint_THTPad_D1.0mm_Drill0.5mm, F.Cu at (155.8, 91.1)
- IC1: renamed from Voltage Divider
- moved D4 0.76 mm to (159.3, 76.7)
- moved R1 0.51 mm to (150.4, 80.5)
Connections:
- R1 pad 1: (no net) -> Sensor_Input_1
- R3 pad 1: (no net) -> Sensor_Input_2
- R5 pad 1: (no net) -> Sensor_Input_4
- R7 pad 1: (no net) -> Sensor_Input_3
Routing:
- net (no net): track 18.6 -> 0.00 mm
- net Sensor_Input_3: track 0.00 -> 5.97 mm
- net Sensor_Input_4: track 0.00 -> 5.76 mm
- net Sensor_Input_1: track 0.00 -> 5.64 mm
- net Sensor_Input_2: track 0.00 -> 5.31 mm
- net Out2: track 4.16 -> 9.24 mm
- net Out3: track 4.14 -> 8.77 mm
- net Out1: track 18.0 -> 19.2 mm
- net Out4: track 16.7 -> 17.4 mm
- added copper zone on F.Cu, net GND
Other:
- board size 24.1 x 21.6 mm -> 21.8 x 17.5 mm
- net class Default: clearance 0.2 -> 0.1
- rule trace_clearance: 0.2 -> 0.1
- rule trace_min: 0.2 -> 0.25
