File: AR20_PDM/PDM_schematic/AR_PDM_v1/PhaseDirect.sch (KiCad schematic (older format))
At the start: 0 parts

Commit message: First draft of Gear phase, shutdown relays, and Direct phases.
Parts:
- added C_bypass? (x2): 0.1uF, symbol AR20_PDM_v1-rescue:C-Device
- added D? (x2): DIODE, symbol AR20_PDM_v1-rescue:DIODE-Simulation_SPICE
- added F? (x2): Fuse, symbol Device:Fuse
- added K? (x2): DIPxx-1Axx-11x, Relay_THT:Relay_StandexMeder_DIP_LowProfile, symbol Relay:DIPxx-1Axx-11x
- added Q? (x2): Q_NJFET_DGS, symbol Device:Q_NJFET_DGS
- added R? (x2): 4.7K, symbol AR20_PDM_v1-rescue:R-Device
- added R? (x2): R_Shunt-Device, symbol AR20_PDM_v1-rescue:R_Shunt-Device
- added U? (x2): INA233, symbol AR20_PDM_v1-rescue:INA233
Connections:
- new net: D?.1 (A), K?.2, Q?.3 (S), Q?.3 (S)
- new net: F?.1, R?.4 (x2)
- new net: F?.2, K?.7, K?.8 (x2)
- new net: R?.2, U?.10 (IN+) (x2)
- new net: R?.3, U?.9 (In-) (x2)
- new net COIL_INJECTOR_OUT: K?.1, K?.14
- new net FP_ENABLE: Q?.2 (G), R?.1
- new net FP_ENABLE_ACM: Q?.2 (G), R?.1
- new net FUEL_PUMP_OUT: K?.1, K?.14
- new net GND: C_bypass?.2, C_bypass?.2, D?.1 (A), K?.2, Q?.1 (D), Q?.1 (D), R?.2, R?.2, U?.1 (A1), U?.1 (A1), U?.2 (A0), U?.2 (A0), U?.7 (GND), U?.7 (GND)
- new net P1_Alert: U?.3 (Alert), U?.3 (Alert)
- new net P1_SDA: U?.4 (SDA), U?.4 (SDA)
- new net P1_SLC: U?.5 (SCL), U?.5 (SCL)
- new net SHUTDOWN_IN: D?.2 (K), D?.2 (K), K?.6, K?.6
- new net VS_12V: R?.1, R?.1
- new net Vs_12v: U?.8 (VBUS), U?.8 (VBUS)
- new net vcc_5v: C_bypass?.1, C_bypass?.1, U?.6 (Vs), U?.6 (Vs)
Other:
- note added: "Close to PIN"
- note added: "Configurable address, \nmust be different for each chip"
