File: AR20_PDM/PDM_schematic/AR_PDM_v1/Phase1.sch (KiCad schematic (older format))
At the start: 18 parts, among them Q1 BTS50025-1TAD, U1 INA233

Commit message: Added label on mosfets, added fuel pump sinking output
Other:
- note added: "Use Logic Level Mosfets. (Gs Threshold <5V)"
Changed lines of the file:
@@
 $Descr A4 11693 8268
 encoding utf-8
-Sheet 6 6
+Sheet 2 6
 Title ""
 Date ""
@@
 AR Path="/5DEB10A1/5DAAC1B1" Ref="R_in?"  Part="1"
 AR Path="/5DEB20EA/5DAAC1B1" Ref="R_in?"  Part="1"
-F 0 "R_in?" V 3093 2400 50  0000 C CNN
+F 0 "R_in" V 3093 2400 50  0000 C CNN
 F 1 "4.7K" V 3184 2400 50  0000 C CNN
 F 2 "" V 3230 2400 50  0001 C CNN
@@
 AR Path="/5DEB10A1/5DAAC1D1" Ref="C_out?"  Part="1"
 AR Path="/5DEB20EA/5DAAC1D1" Ref="C_out?"  Part="1"
-F 0 "C_out?" H 4915 2896 50  0000 L CNN
+F 0 "C_out" H 4915 2896 50  0000 L CNN
 F 1 "220nf" H 4915 2805 50  0000 L CNN
 F 2 "" H 4838 2700 50  0001 C CNN
@@
 AR Path="/5DEB10A1/5DAAC1D7" Ref="C_in?"  Part="1"
 AR Path="/5DEB20EA/5DAAC1D7" Ref="C_in?"  Part="1"
-F 0 "C_in?" H 3615 1996 50  0000 L CNN
+F 0 "C_in" H 3615 1996 50  0000 L CNN
 F 1 "220nf" H 3615 1905 50  0000 L CNN
 F 2 "" H 3538 1800 50  0001 C CNN
@@
 AR Path="/5DEB10A1/5DAAC201" Ref="C_bypass?"  Part="1"
 AR Path="/5DEB20EA/5DAAC201" Ref="C_bypass?"  Part="1"
-F 0 "C_bypass?" V 8248 3350 50  0000 C CNN
+F 0 "C_bypass" V 8248 3350 50  0000 C CNN
 F 1 "0.1uF" V 8339 3350 50  0000 C CNN
 F 2 "" H 8538 3200 50  0001 C CNN
@@
 AR Path="/5DEB10A1/5DAAC252" Ref="R_IS?"  Part="1"
 AR Path="/5DEB20EA/5DAAC252" Ref="R_IS?"  Part="1"
-F 0 "R_IS?" V 3475 3500 50  0000 C CNN
+F 0 "R_IS" V 3475 3500 50  0000 C CNN
 F 1 "53R_0.1%" V 3566 3500 50  0000 C CNN
 F 2 "" V 3630 3500 50  0001 C CNN
@@
 AR Path="/5DEB10A1/5DAAC283" Ref="C_sense?"  Part="1"
 AR Path="/5DEB20EA/5DAAC283" Ref="C_sense?"  Part="1"
-F 0 "C_sense?" H 3265 3546 50  0000 L CNN
+F 0 "C_sense" H 3265 3546 50  0000 L CNN
 F 1 "10nf" H 3265 3455 50  0000 L CNN
 F 2 "" H 3188 3350 50  0001 C CNN
@@
 AR Path="/5DEB10A1/5DA8B874" Ref="Q?"  Part="1"
 AR Path="/5DEB20EA/5DA8B874" Ref="Q?"  Part="1"
-F 0 "Q?" H 4255 3215 50  0000 C CNN
+F 0 "Q1" H 4255 3215 50  0000 C CNN
 F 1 "BTS50025-1TAD" H 4255 3124 50  0000 C CNN
 F 2 "" H 4250 2650 50  0001 C CNN
@@
 AR Path="/5DEB10A1/5DA8DC6C" Ref="U?"  Part="1"
 AR Path="/5DEB20EA/5DA8DC6C" Ref="U?"  Part="1"
-F 0 "U?" H 9225 4465 50  0000 C CNN
+F 0 "U1" H 9225 4465 50  0000 C CNN
 F 1 "INA233" H 9225 4374 50  0000 C CNN
 F 2 "" H 9200 4050 50  0001 C CNN
@@
 AR Path="/5DEB10A1/5DAE255C" Ref="C_vs?"  Part="1"
 AR Path="/5DEB20EA/5DAE255C" Ref="C_vs?"  Part="1"
-F 0 "C_vs?" H 5315 2046 50  0000 L CNN
+F 0 "C_vs" H 5315 2046 50  0000 L CNN
 F 1 "100nf" H 5315 1955 50  0000 L CNN
 F 2 "" H 5238 1850 50  0001 C CNN
@@
 Wire Wire Line
 	6300 1900 6300 2000
+Text Notes 1075 2725 0    50   ~ 0
+Use Logic Level Mosfets. (Gs Threshold <5V)
 $EndSCHEMATC

Commit message: Major update to testcode
- Set up for visual studio code
- Re organized structure
- created INA233 objects
- Made object oriented structure
Connections:
- wire segments 71 -> 73
Changed lines of the file:
@@
 	1    0    0    -1
 $EndComp
-Text HLabel 8350 4100 0    50   Input ~ 10
-Vs_12v
 Text HLabel 8750 2850 1    50   Input ~ 10
 vcc_5v
@@
 Wire Wire Line
 	3700 3100 3700 3300
-Wire Wire Line
-	8750 4100 8350 4100
 Text HLabel 4650 1600 0    50   Input ~ 10
 Vs_12v
@@
 Wire Wire Line
 	5400 2550 5400 2775
-Wire Wire Line
-	5400 2775 6950 2775
 Connection ~ 4800 2550
 Wire Wire Line
@@
 Text Notes 1075 2725 0    50   ~ 0
 Use Logic Level Mosfets. (Gs Threshold <5V)
+Wire Wire Line
+	6000 4100 6000 2775
+Wire Wire Line
+	6000 4100 8750 4100
+Wire Wire Line
+	5400 2775 6000 2775
+Wire Wire Line
+	6000 2775 6950 2775
+Connection ~ 6000 2775
 $EndSCHEMATC
