File: AR20_PDM/PDM_schematic/AR_PDM_v1/Phase1.sch (KiCad schematic (older format))
At the start: 12 parts, among them Q1 BTS50025-1TAD, U5 INA233

Commit message: Alpha version DONE! - Gerber files generated
- Tweeked
- checked and re cheked
- added all missing components
- Created a really nice silkscreen
- Ready To Test
Parts:
- renumbered R3 to R4, R4 to R5, R5 to R6, R6 to R7, R_Shunt4 to R8, U5 to U2
Changed lines of the file:
@@
 $EndDescr
 $Comp
-L AR20_PDM_v1-rescue:R-Device R4
+L AR20_PDM_v1-rescue:R-Device R5
 U 1 1 5E21B807
 P 3300 2400
-AR Path="/5DA89415/5E21B807" Ref="R4"  Part="1"
+AR Path="/5DA89415/5E21B807" Ref="R5"  Part="1"
 AR Path="/5DEB10A1/5E21B807" Ref="R?"  Part="1"
 AR Path="/5DEB20EA/5E21B807" Ref="R?"  Part="1"
@@
 AR Path="/5E0FDCCC/5E21B807" Ref="R?"  Part="1"
 AR Path="/5E10174B/5E21B807" Ref="R?"  Part="1"
-F 0 "R4" V 3093 2400 50  0000 C CNN
+F 0 "R5" V 3093 2400 50  0000 C CNN
 F 1 "4k7" V 3184 2400 50  0000 C CNN
 F 2 "Resistor_SMD:R_0603_1608Metric" V 3230 2400 50  0001 C CNN
@@
 $EndComp
 $Comp
-L AR20_PDM_v1-rescue:R-Device R3
+L AR20_PDM_v1-rescue:R-Device R4
 U 1 1 5E21B81B
 P 2250 1850
-AR Path="/5DA89415/5E21B81B" Ref="R3"  Part="1"
+AR Path="/5DA89415/5E21B81B" Ref="R4"  Part="1"
 AR Path="/5DEB10A1/5E21B81B" Ref="R?"  Part="1"
 AR Path="/5DEB20EA/5E21B81B" Ref="R?"  Part="1"
@@
 AR Path="/5E0FDCCC/5E21B81B" Ref="R?"  Part="1"
 AR Path="/5E10174B/5E21B81B" Ref="R?"  Part="1"
-F 0 "R3" H 2320 1896 50  0000 L CNN
+F 0 "R4" H 2320 1896 50  0000 L CNN
 F 1 "4k7" H 2320 1805 50  0000 L CNN
 F 2 "Resistor_SMD:R_0603_1608Metric" V 2180 1850 50  0001 C CNN
@@
 	4800 2550 4800 2700
 $Comp
-L AR20_PDM_v1-rescue:GND-power #PWR033
+L AR20_PDM_v1-rescue:GND-power #PWR025
 U 1 1 5E21B82A
 P 8300 3550
-AR Path="/5DA89415/5E21B82A" Ref="#PWR033"  Part="1"
+AR Path="/5DA89415/5E21B82A" Ref="#PWR025"  Part="1"
 AR Path="/5DEB10A1/5E21B82A" Ref="#PWR?"  Part="1"
 AR Path="/5DEB20EA/5E21B82A" Ref="#PWR?"  Part="1"
@@
 AR Path="/5E0FDCCC/5E21B82A" Ref="#PWR?"  Part="1"
 AR Path="/5E10174B/5E21B82A" Ref="#PWR?"  Part="1"
-F 0 "#PWR033" H 8300 3300 50  0001 C CNN
+F 0 "#PWR025" H 8300 3300 50  0001 C CNN
 F 1 "GND" V 8305 3422 50  0000 R CNN
 F 2 "" H 8300 3550 50  0001 C CNN
@@
 	9700 3950 10350 3950
 $Comp
-L AR20_PDM_v1-rescue:GND-power #PWR034
+L AR20_PDM_v1-rescue:GND-power #PWR026
 U 1 1 5E21B833
 P 9200 5150
-AR Path="/5DA89415/5E21B833" Ref="#PWR034"  Part="1"
+AR Path="/5DA89415/5E21B833" Ref="#PWR026"  Part="1"
 AR Path="/5DEB10A1/5E21B833" Ref="#PWR?"  Part="1"
 AR Path="/5DEB20EA/5E21B833" Ref="#PWR?"  Part="1"
@@
 AR Path="/5E0FDCCC/5E21B833" Ref="#PWR?"  Part="1"
 AR Path="/5E10174B/5E21B833" Ref="#PWR?"  Part="1"
-F 0 "#PWR034" H 9200 4900 50  0001 C CNN
+F 0 "#PWR026" H 9200 4900 50  0001 C CNN
 F 1 "GND" H 9205 4977 50  0000 C CNN
 F 2 "" H 9200 5150 50  0001 C CNN
@@
 $EndComp
 $Comp
-L AR20_PDM_v1-rescue:GND-power #PWR030
+L AR20_PDM_v1-rescue:GND-power #PWR022
 U 1 1 5E21B839
 P 4800 3000
-AR Path="/5DA89415/5E21B839" Ref="#PWR030"  Part="1"
+AR Path="/5DA89415/5E21B839" Ref="#PWR022"  Part="1"
 AR Path="/5DEB10A1/5E21B839" Ref="#PWR?"  Part="1"
 AR Path="/5DEB20EA/5E21B839" Ref="#PWR?"  Part="1"
@@
 AR Path="/5E0FDCCC/5E21B839" Ref="#PWR?"  Part="1"
 AR Path="/5E10174B/5E21B839" Ref="#PWR?"  Part="1"
-F 0 "#PWR030" H 4800 2750 50  0001 C CNN
+F 0 "#PWR022" H 4800 2750 50  0001 C CNN
 F 1 "GND" H 4805 2827 50  0000 C CNN
 F 2 "" H 4800 3000 50  0001 C CNN
@@
 $EndComp
 $Comp
-L AR20_PDM_v1-rescue:GND-power #PWR029
+L AR20_PDM_v1-rescue:GND-power #PWR021
 U 1 1 5E21B83C
 P 4250 2800
-AR Path="/5DA89415/5E21B83C" Ref="#PWR029"  Part="1"
+AR Path="/5DA89415/5E21B83C" Ref="#PWR021"  Part="1"
 AR Path="/5DEB10A1/5E21B83C" Ref="#PWR?"  Part="1"
 AR Path="/5DEB20EA/5E21B83C" Ref="#PWR?"  Part="1"
@@
 AR Path="/5E0FDCCC/5E21B83C" Ref="#PWR?"  Part="1"
 AR Path="/5E10174B/5E21B83C" Ref="#PWR?"  Part="1"
-F 0 "#PWR029" H 4250 2550 50  0001 C CNN
+F 0 "#PWR021" H 4250 2550 50  0001 C CNN
 F 1 "GND" H 4255 2627 50  0000 C CNN
 F 2 "" H 4250 2800 50  0001 C CNN
@@
 $EndComp
 $Comp
-L AR20_PDM_v1-rescue:GND-power #PWR027
+L AR20_PDM_v1-rescue:GND-power #PWR020
 U 1 1 5E21B845
 P 3500 1800
-AR Path="/5DA89415/5E21B845" Ref="#PWR027"  Part="1"
+AR Path="/5DA89415/5E21B845" Ref="#PWR020"  Part="1"
 AR Path="/5DEB10A1/5E21B845" Ref="#PWR?"  Part="1"
 AR Path="/5DEB20EA/5E21B845" Ref="#PWR?"  Part="1"
@@
 AR Path="/5E0FDCCC/5E21B845" Ref="#PWR?"  Part="1"
 AR Path="/5E10174B/5E21B845" Ref="#PWR?"  Part="1"
-F 0 "#PWR027" H 3500 1550 50  0001 C CNN
+F 0 "#PWR020" H 3500 1550 50  0001 C CNN
 F 1 "GND" H 3505 1627 50  0000 C CNN
 F 2 "" H 3500 1800 50  0001 C CNN
@@
 $EndComp
 $Comp
-L AR20_PDM_v1-rescue:INA233 U5
+L AR20_PDM_v1-rescue:INA233 U2
 U 1 1 5E21B805
 P 9200 4050
-AR Path="/5DA89415/5E21B805" Ref="U5"  Part="1"
+AR Path="/5DA89415/5E21B805" Ref="U2"  Part="1"
 AR Path="/5DEB10A1/5E21B805" Ref="U?"  Part="1"
 AR Path="/5DEB20EA/5E21B805" Ref="U?"  Part="1"
@@
 AR Path="/5E0FDCCC/5E21B805" Ref="U?"  Part="1"
 AR Path="/5E10174B/5E21B805" Ref="U?"  Part="1"
-F 0 "U5" H 9225 4465 50  0000 C CNN
+F 0 "U2" H 9225 4465 50  0000 C CNN
 F 1 "INA233" H 9225 4374 50  0000 C CNN
 F 2 "AR_PDM_v1:INA233" H 9200 4050 50  0001 C CNN
@@
 Close to PIN
 $Comp
-L AR20_PDM_v1-rescue:GND-power #PWR031
+L AR20_PDM_v1-rescue:GND-power #PWR023
 U 1 1 5E21B85C
 P 5200 2150
-AR Path="/5DA89415/5E21B85C" Ref="#PWR031"  Part="1"
+AR Path="/5DA89415/5E21B85C" Ref="#PWR023"  Part="1"
 AR Path="/5DEB10A1/5E21B85C" Ref="#PWR?"  Part="1"
 AR Path="/5DEB20EA/5E21B85C" Ref="#PWR?"  Part="1"
@@
 AR Path="/5E0FDCCC/5E21B85C" Ref="#PWR?"  Part="1"
 AR Path="/5E10174B/5E21B85C" Ref="#PWR?"  Part="1"
-F 0 "#PWR031" H 5200 1900 50  0001 C CNN
+F 0 "#PWR023" H 5200 1900 50  0001 C CNN
 F 1 "GND" H 5205 1977 50  0000 C CNN
 F 2 "" H 5200 2150 50  0001 C CNN
@@
 $EndComp
 $Comp
-L AR20_PDM_v1-rescue:GND-power #PWR032
+L AR20_PDM_v1-rescue:GND-power #PWR024
 U 1 1 5E21B866
 P 5800 2300
-AR Path="/5DA89415/5E21B866" Ref="#PWR032"  Part="1"
+AR Path="/5DA89415/5E21B866" Ref="#PWR024"  Part="1"
 AR Path="/5DEB10A1/5E21B866" Ref="#PWR?"  Part="1"
 AR Path="/5DEB20EA/5E21B866" Ref="#PWR?"  Part="1"
@@
 AR Path="/5E0FDCCC/5E21B866" Ref="#PWR?"  Part="1"
 AR Path="/5E10174B/5E21B866" Ref="#PWR?"  Part="1"
-F 0 "#PWR032" H 5800 2050 50  0001 C CNN
+F 0 "#PWR024" H 5800 2050 50  0001 C CNN
 F 1 "GND" H 5805 2127 50  0000 C CNN
 F 2 "" H 5800 2300 50  0001 C CNN
@@
 $EndComp
 $Comp
-L AR20_PDM_v1-rescue:R-Device R6
+L AR20_PDM_v1-rescue:R-Device R7
 U 1 1 5E21B870
 P 5800 1750
-AR Path="/5DA89415/5E21B870" Ref="R6"  Part="1"
+AR Path="/5DA89415/5E21B870" Ref="R7"  Part="1"
 AR Path="/5DEB10A1/5E21B870" Ref="R?"  Part="1"
 AR Path="/5DEB20EA/5E21B870" Ref="R?"  Part="1"
@@
 AR Path="/5E0FDCCC/5E21B870" Ref="R?"  Part="1"
 AR Path="/5E10174B/5E21B870" Ref="R?"  Part="1"
-F 0 "R6" V 5593 1750 50  0000 C CNN
+F 0 "R7" V 5593 1750 50  0000 C CNN
 F 1 "3.9R" V 5684 1750 50  0000 C CNN
 F 2 "Resistor_SMD:R_0603_1608Metric" V 5730 1750 50  0001 C CNN
@@
 	6000 4100 8750 4100
 $Comp
-L AR20_PDM_v1-rescue:R-Device R5
+L AR20_PDM_v1-rescue:R-Device R6
 U 1 1 5E21B875
 P 3700 3450
-AR Path="/5DA89415/5E21B875" Ref="R5"  Part="1"
+AR Path="/5DA89415/5E21B875" Ref="R6"  Part="1"
 AR Path="/5DEB10A1/5E21B875" Ref="R?"  Part="1"
 AR Path="/5DEB20EA/5E21B875" Ref="R?"  Part="1"
@@
 AR Path="/5E0FDCCC/5E21B875" Ref="R?"  Part="1"
 AR Path="/5E10174B/5E21B875" Ref="R?"  Part="1"
-F 0 "R5" H 3770 3496 50  0000 L CNN
+F 0 "R6" H 3770 3496 50  0000 L CNN
 F 1 "4k7" H 3770 3405 50  0000 L CNN
 F 2 "Resistor_SMD:R_0603_1608Metric" V 3630 3450 50  0001 C CNN
@@
 	6325 2950 6325 4400
 $Comp
-L AR20_PDM_v1-rescue:R-Device R_Shunt4
+L AR20_PDM_v1-rescue:R-Device R8
 U 1 1 5E1C5925
 P 6475 2950
-AR Path="/5DA89415/5E1C5925" Ref="R_Shunt4"  Part="1"
-AR Path="/5DEB10A1/5E1C5925" Ref="R_Shunt?"  Part="1"
-AR Path="/5DEB20EA/5E1C5925" Ref="R_Shunt?"  Part="1"
-AR Path="/5E0E4725/5E1C5925" Ref="R_Shunt?"  Part="1"
-AR Path="/5E0E4A93/5E1C5925" Ref="R_Shunt?"  Part="1"
-AR Path="/5E0E4EB5/5E1C5925" Ref="R_Shunt?"  Part="1"
-AR Path="/5E0E5304/5E1C5925" Ref="R_Shunt?"  Part="1"
-AR Path="/5E0E594B/5E1C5925" Ref="R_Shunt?"  Part="1"
-AR Path="/5E0E607C/5E1C5925" Ref="R_Shunt?"  Part="1"
-AR Path="/5E0FB5C8/5E1C5925" Ref="R_Shunt?"  Part="1"
-AR Path="/5E0FBBBD/5E1C5925" Ref="R_Shunt?"  Part="1"
-AR Path="/5E0FC3A2/5E1C5925" Ref="R_Shunt?"  Part="1"
-AR Path="/5E0FCFDC/5E1C5925" Ref="R_Shunt?"  Part="1"
-AR Path="/5E0FDCCC/5E1C5925" Ref="R_Shunt?"  Part="1"
-AR Path="/5E10174B/5E1C5925" Ref="R_Shunt?"  Part="1"
-F 0 "R_Shunt4" V 6268 2950 50  0000 C CNN
+AR Path="/5DA89415/5E1C5925" Ref="R8"  Part="1"
+AR Path="/5DEB10A1/5E1C5925" Ref="R?"  Part="1"
+AR Path="/5DEB20EA/5E1C5925" Ref="R?"  Part="1"
+AR Path="/5E0E4725/5E1C5925" Ref="R?"  Part="1"
+AR Path="/5E0E4A93/5E1C5925" Ref="R?"  Part="1"
+AR Path="/5E0E4EB5/5E1C5925" Ref="R?"  Part="1"
+AR Path="/5E0E5304/5E1C5925" Ref="R?"  Part="1"
+AR Path="/5E0E594B/5E1C5925" Ref="R?"  Part="1"
+AR Path="/5E0E607C/5E1C5925" Ref="R?"  Part="1"
+AR Path="/5E0FB5C8/5E1C5925" Ref="R?"  Part="1"
+AR Path="/5E0FBBBD/5E1C5925" Ref="R?"  Part="1"
+AR Path="/5E0FC3A2/5E1C5925" Ref="R?"  Part="1"
+AR Path="/5E0FCFDC/5E1C5925" Ref="R?"  Part="1"
+AR Path="/5E0FDCCC/5E1C5925" Ref="R?"  Part="1"
+AR Path="/5E10174B/5E1C5925" Ref="R?"  Part="1"
+F 0 "R8" V 6268 2950 50  0000 C CNN
 F 1 "2m_1%_4W" V 6359 2950 50  0000 C CNN
 F 2 "Resistor_SMD:R_2512_6332Metric" V 6405 2950 50  0001 C CNN
