File: AR20_PDM/PDM_schematic/AR_PDM_v1/AR20_PDM_v1.sch (KiCad schematic (older format))
At the start: 14 parts, among them J1 High_Curret_terminal, J2 1-776163-1, U1 ACM_2020

Commit message: PCB Design, Work in progress
Connections:
- net CLUTCH_ACT_OUT: now also J2.12
- net COIL_INJECTOR_OUT: now also J2.13
- net ETC_OUT: now also J2.11
- net FUEL_PUMP_OUT: now also J2.24
- net GND: now also J2.20, J2.21, J2.22, J2.9
- net IGN_SWITCH_OUT: now also J2.23
- net MCU_UNITS_FEED_OUT: now also J2.10
- net P1_EN_AUX: now also J2.27
- net P2_EN_AUX: now also J2.16
- net P3_EN_AUX: now also J2.28
- net P4_EN_AUX: now also J2.17
- net P5_EN_AUX: now also J2.29
- net P6_EN_AUX: now also J2.18
- net P7_EN_AUX: now also J2.19
- net SHUTDOWN_IN: now also J2.14
- net SHUTDOWN_OUT: now also J2.35
Changed lines of the file:
@@
 vcc_5v
-$Sheet
-S 8450 700  1550 725
-U 5DA8920B
-F0 "Fuel_Ignition_ShutdownCircuit" 50
-F1 "Fuel_Ignition_Shutdown.sch" 50
-F2 "vcc_5v" I L 8450 950 50
-F3 "SHUTDOWN_IN" I L 8450 750 50
-F4 "FP_Alert" O L 8450 1275 50
-F5 "SDA" B L 8450 1075 50
-F6 "SLC" I L 8450 1175 50
-F7 "COIL_INJECTOR_Alert" O L 8450 1375 50
-F8 "V+12V" I L 8450 850 50
-F9 "FUEL_PUMP_OUT" O R 10000 875 50
-F10 "FP_ENABLE_ACM" I R 10000 975 50
-F11 "COIL_INJECTOR_OUT" O R 10000 750 50
-F12 "FP_ENABLE_AUX" I R 10000 1075 50
-F13 "FP_ENABLE_RELAY_SINK" O R 10000 1175 50
-F14 "ACM_Shutdown_Circuit" I R 10000 1275 50
-$EndSheet
 $Sheet
 S 8475 1650 1500 525
@@
 SHUTDOWN_IN
 Text GLabel 4375 2050 0    50   Input ~ 0
-P7_OUT
+P7_Shunt
 Text GLabel 4375 1950 0    50   Input ~ 0
-P6_OUT
+P6_Shunt
 Text GLabel 4375 1850 0    50   Input ~ 0
-P5_OUT
+P5_Shunt
 Text GLabel 4375 1750 0    50   Input ~ 0
-P4_OUT
+P4_Shunt
 Text GLabel 4375 1650 0    50   Input ~ 0
-P3_OUT
+P3_Shunt
 Text GLabel 4375 1550 0    50   Input ~ 0
-P2_OUT
+P2_Shunt
 Text GLabel 4375 1450 0    50   Input ~ 0
-P1_OUT
+P1_Shunt
 Text GLabel 4375 2800 0    50   Input ~ 0
 COIL_INJECTOR_OUT
@@
 Text GLabel 12750 1275 0    50   Input ~ 0
 P7_EN_ACM
-Text GLabel 13450 6825 1    50   Input ~ 0
+Text GLabel 9475 7875 1    50   Input ~ 0
 P3_EN_AUX
 Text GLabel 5825 2325 2    50   Input ~ 0
@@
 Loss of power, flyback protection. \nPlace relativly near all of the mosfets.
 Wire Wire Line
-	12950 8175 12950 8375
+	11775 7675 11775 7875
 Text GLabel 14050 6825 1    50   Input ~ 0
 CAN_LOW
 Text GLabel 13950 6825 1    50   Input ~ 0
 CAN_HIGH
-Text GLabel 13650 6825 1    50   Input ~ 0
+Text GLabel 9375 7875 1    50   Input ~ 0
 P5_EN_AUX
-Text GLabel 13750 6825 1    50   Input ~ 0
+Text GLabel 10675 7875 1    50   Input ~ 0
 P6_EN_AUX
 Text GLabel 14300 1875 2    50   Input ~ 0
 P3_EN_ACM
-Text GLabel 13250 6825 1    50   Input ~ 0
+Text GLabel 9575 7875 1    50   Input ~ 0
 P1_EN_AUX
-Text GLabel 13550 6825 1    50   Input ~ 0
+Text GLabel 10775 7875 1    50   Input ~ 0
 P4_EN_AUX
-Text GLabel 13350 6825 1    50   Input ~ 0
+Text GLabel 10875 7875 1    50   Input ~ 0
 P2_EN_AUX
-Text GLabel 13850 6825 1    50   Input ~ 0
+Text GLabel 10575 7875 1    50   Input ~ 0
 P7_EN_AUX
-Text GLabel 13150 6825 1    50   Input ~ 0
+Text GLabel 12125 6775 1    50   Input ~ 0
 FP_ENABLE_AUX
-Text GLabel 13050 6825 1    50   Input ~ 0
-FP_ENABLE_RELAY_SINK
-Text GLabel 13050 8400 1    50   Input ~ 0
-GEAR_ACT_COIL_GND
-Text GLabel 14350 8400 1    50   Input ~ 0
+Text GLabel 11675 7875 1    50   Input ~ 0
 MCU_UNITS_FEED_OUT
-Text GLabel 14250 8400 1    50   Input ~ 0
+Text GLabel 10175 7875 1    50   Input ~ 0
 IGN_SWITCH_OUT
-Text GLabel 14150 8400 1    50   Input ~ 0
+Text GLabel 11575 7875 1    50   Input ~ 0
 ETC_OUT
-Text GLabel 14050 8400 1    50   Input ~ 0
+Text GLabel 11475 7875 1    50   Input ~ 0
 CLUTCH_ACT_OUT
-Text GLabel 13950 8400 1    50   Input ~ 0
+Text GLabel 9875 7875 1    50   Input ~ 0
 FUEL_PUMP_OUT
-Text GLabel 13850 8400 1    50   Input ~ 0
+Text GLabel 11175 7875 1    50   Input ~ 0
 COIL_INJECTOR_OUT
-Text GLabel 13150 8400 1    50   Input ~ 0
+Text GLabel 13300 7750 1    50   Input ~ 0
 P1_OUT
-Text GLabel 13250 8400 1    50   Input ~ 0
+Text GLabel 13400 7750 1    50   Input ~ 0
 P2_OUT
-Text GLabel 13350 8400 1    50   Input ~ 0
+Text GLabel 13500 7750 1    50   Input ~ 0
 P3_OUT
-Text GLabel 13450 8400 1    50   Input ~ 0
+Text GLabel 13600 7750 1    50   Input ~ 0
 P4_OUT
-Text GLabel 13550 8400 1    50   Input ~ 0
+Text GLabel 13700 7750 1    50   Input ~ 0
 P5_OUT
-Text GLabel 13650 8400 1    50   Input ~ 0
+Text GLabel 13800 7750 1    50   Input ~ 0
 P6_OUT
-Text GLabel 13750 8400 1    50   Input ~ 0
+Text GLabel 13900 7750 1    50   Input ~ 0
 P7_OUT
 $Comp
 L AR20_PDM_v1-rescue:GND-power #PWR?
 U 1 1 5E117EF0
-P 12950 8175
+P 11775 7675
 AR Path="/5DA89415/5E117EF0" Ref="#PWR?"  Part="1"
 AR Path="/5DA8920B/5E117EF0" Ref="#PWR?"  Part="1"
 AR Path="/5DE4D361/5E117EF0" Ref="#PWR?"  Part="1"
 AR Path="/5E117EF0" Ref="#PWR09"  Part="1"
-F 0 "#PWR09" H 12950 7925 50  0001 C CNN
-F 1 "GND" H 12955 8002 50  0000 C CNN
-F 2 "" H 12950 8175 50  0001 C CNN
-F 3 "" H 12950 8175 50  0001 C CNN
-	1    12950 8175
+F 0 "#PWR09" H 11775 7425 50  0001 C CNN
+F 1 "GND" H 11780 7502 50  0000 C CNN
+F 2 "" H 11775 7675 50  0001 C CNN
+F 3 "" H 11775 7675 50  0001 C CNN
+	1    11775 7675
 	-1   0    0    1
 $EndComp
@@
 F21 "P2_EN_ACM" I R 5825 1650 50
 F22 "P1_EN_ACM" I R 5825 1550 50
-F23 "P1_OUT" I L 4375 1450 50
-F24 "SHUTDOWN_IN" I L 4375 2175 50
-F25 "COIL_INJECTOR_OUT" I L 4375 2800 50
-F26 "FUEL_PUMP_OUT" I L 4375 2900 50
-F27 "CLUTCH_ACT_OUT" I L 4375 2600 50
-F28 "ETC_OUT" I L 4375 2700 50
-F29 "SHUTDOWN_OUT" I L 4375 2275 50
-F30 "IGN_SWITCH_OUT" I L 4375 2500 50
-F31 "MCU_UNITS_FEED_OUT" I L 4375 2400 50
-F32 "Switch" I R 5825 3050 50
-F33 "vcc_5v" I R 5825 3150 50
-F34 "V+12V" I R 5825 3250 50
-F35 "P2_OUT" I L 4375 1550 50
-F36 "P3_OUT" I L 4375 1650 50
-F37 "P4_OUT" I L 4375 1750 50
-F38 "P5_OUT" I L 4375 1850 50
-F39 "P6_OUT" I L 4375 1950 50
-F40 "P7_OUT" I L 4375 2050 50
-F41 "P1_Fault" O R 5825 2325 50
-F42 "P2_Fault" O R 5825 2425 50
-F43 "P3_Fault" O R 5825 2525 50
-F44 "P4_Fault" O R 5825 2625 50
-F45 "P5_Fault" O R 5825 2725 50
-F46 "P6_Fault" O R 5825 2825 50
-F47 "P7_Fault" O R 5825 2925 50
-F48 "COIL_INJ_Fault" O L 4375 3150 50
-F49 "FP_Fault" O L 4375 3250 50
+F23 "COIL_INJECTOR_OUT" I L 4375 2800 50
+F24 "FUEL_PUMP_OUT" I L 4375 2900 50
+F25 "CLUTCH_ACT_OUT" I L 4375 2600 50
+F26 "ETC_OUT" I L 4375 2700 50
+F27 "SHUTDOWN_OUT" I L 4375 2275 50
+F28 "IGN_SWITCH_OUT" I L 4375 2500 50
+F29 "MCU_UNITS_FEED_OUT" I L 4375 2400 50
+F30 "Switch" I R 5825 3050 50
+F31 "vcc_5v" I R 5825 3150 50
+F32 "V+12V" I R 5825 3250 50
+F33 "P1_Fault" O R 5825 2325 50
+F34 "P2_Fault" O R 5825 2425 50
+F35 "P3_Fault" O R 5825 2525 50
+F36 "P4_Fault" O R 5825 2625 50
+F37 "P5_Fault" O R 5825 2725 50
+F38 "P6_Fault" O R 5825 2825 50
+F39 "P7_Fault" O R 5825 2925 50
+F40 "COIL_INJ_Fault" O L 4375 3150 50
+F41 "FP_Fault" O L 4375 3250 50
+F42 "Shutdown_Led" I L 4375 2175 50
+F43 "SHUTDOWN_IN" I L 4375 3025 50
+F44 "P2_Shunt" I L 4375 1550 50
+F45 "P3_Shunt" I L 4375 1650 50
+F46 "P4_Shunt" I L 4375 1750 50
+F47 "P5_Shunt" I L 4375 1850 50
+F48 "P6_Shunt" I L 4375 1950 50
+F49 "P7_Shunt" I L 4375 2050 50
+F50 "P1_Shunt" I L 4375 1450 50
 $EndSheet
-Text GLabel 4375 2175 0    50   Input ~ 0
-SHUTDOWN_IN
 Text GLabel 4375 2275 0    50   Input ~ 0
 SHUTDOWN_OUT
@@
 Wire Notes Line
 	5925 7650 5925 6750
-Text GLabel 14450 8400 1    50   Input ~ 0
+Text GLabel 8775 7875 1    50   Input ~ 0
 SHUTDOWN_OUT
 Text Notes 13850 7050 0    50   Italic 10
@@
 	-1   0    0    1
 $EndComp
-Text GLabel 14150 6825 1    50   Input ~ 0
-GND_Low_Power
 Text GLabel 14450 6825 1    50   Input ~ 0
 RX
@@
 Text GLabel 14650 6825 1    50   Input ~ 0
 P6_GearA_open_drain_output
-Text GLabel 14350 6825 1    50   Input ~ 0
+Text GLabel 11075 7875 1    50   Input ~ 0
 SHUTDOWN_IN
-Text GLabel 14250 6825 1    50   Input ~ 0
-GND_Low_Power
 $Comp
 L AR20_PDM_v1-rescue:1-776163-1 J2
@@
 NoConn ~ 12750 2625
 NoConn ~ 12750 2925
+$Sheet
+S 8450 700  1550 725
+U 5DA8920B
+F0 "Fuel_Ignition_ShutdownCircuit" 50
+F1 "Fuel_Ignition_Shutdown.sch" 50
+F2 "vcc_5v" I L 8450 950 50
+F3 "SHUTDOWN_IN" I L 8450 750 50
+F4 "FP_Alert" O L 8450 1275 50
+F5 "SDA" B L 8450 1075 50
+F6 "SLC" I L 8450 1175 50
+F7 "COIL_INJECTOR_Alert" O L 8450 1375 50
+F8 "V+12V" I L 8450 850 50
+F9 "FUEL_PUMP_OUT" O R 10000 875 50
+F10 "FP_ENABLE_ACM" I R 10000 975 50
+F11 "COIL_INJECTOR_OUT" O R 10000 750 50
+F12 "FP_ENABLE_AUX" I R 10000 1075 50
+F13 "FP_ENABLE_RELAY_SINK" O R 10000 1175 50
+F14 "ACM_Shutdown_Circuit" I R 10000 1275 50
+F15 "SHUTDOWN_Led" O R 10000 1375 50
+$EndSheet
+Text GLabel 11875 6850 1    50   Input ~ 0
+FP_ENABLE_RELAY_SINK
+Wire Wire Line
+	10000 1375 10100 1375
+Text GLabel 10100 1375 2    50   Input ~ 0
+Shutdown_Led
+Text GLabel 4375 2175 0    50   Input ~ 0
+Shutdown_Led
+Text GLabel 4375 3025 0    50   Input ~ 0
+SHUTDOWN_IN
+$Comp
+L AR20_PDM_v1-rescue:GND-power #PWR?
+U 1 1 5E2C8E2C
+P 10275 7675
+AR Path="/5DA89415/5E2C8E2C" Ref="#PWR?"  Part="1"
+AR Path="/5DA8920B/5E2C8E2C" Ref="#PWR?"  Part="1"
+AR Path="/5DE4D361/5E2C8E2C" Ref="#PWR?"  Part="1"
+AR Path="/5E2C8E2C" Ref="#PWR0136"  Part="1"
+F 0 "#PWR0136" H 10275 7425 50  0001 C CNN
+F 1 "GND" H 10280 7502 50  0000 C CNN
+F 2 "" H 10275 7675 50  0001 C CNN
+F 3 "" H 10275 7675 50  0001 C CNN
+	1    10275 7675
+	-1   0    0    1
+$EndComp
+Wire Wire Line
+	10275 7675 10275 7875
+$Comp
+L AR20_PDM_v1-rescue:GND-power #PWR?
+U 1 1 5E2C5A37
+P 10375 7675
+AR Path="/5DA89415/5E2C5A37" Ref="#PWR?"  Part="1"
+AR Path="/5DA8920B/5E2C5A37" Ref="#PWR?"  Part="1"
+AR Path="/5DE4D361/5E2C5A37" Ref="#PWR?"  Part="1"
+AR Path="/5E2C5A37" Ref="#PWR0135"  Part="1"
+F 0 "#PWR0135" H 10375 7425 50  0001 C CNN
+F 1 "GND" H 10380 7502 50  0000 C CNN
+F 2 "" H 10375 7675 50  0001 C CNN
+F 3 "" H 10375 7675 50  0001 C CNN
+	1    10375 7675
+	-1   0    0    1
+$EndComp
+Wire Wire Line
+	10375 7675 10375 7875
+$Comp
+L AR20_PDM_v1-rescue:GND-power #PWR?
+U 1 1 5E2BF009
+P 10475 7675
+AR Path="/5DA89415/5E2BF009" Ref="#PWR?"  Part="1"
+AR Path="/5DA8920B/5E2BF009" Ref="#PWR?"  Part="1"
+AR Path="/5DE4D361/5E2BF009" Ref="#PWR?"  Part="1"
+AR Path="/5E2BF009" Ref="#PWR0134"  Part="1"
+F 0 "#PWR0134" H 10475 7425 50  0001 C CNN
+F 1 "GND" H 10480 7502 50  0000 C CNN
+F 2 "" H 10475 7675 50  0001 C CNN
+F 3 "" H 10475 7675 50  0001 C CNN
+	1    10475 7675
+	-1   0    0    1
+$EndComp
+Wire Wire Line
+	10475 7675 10475 7875
 $EndSCHEMATC

Commit message: PCB Design,  minor schematics changes, work in progress, see description
- Removed mos sense caps and resistors accept one, 
since only one measurement can be done, at a time.
- added mos sens protection resistors on each line, to protect mux mosfets and micro controller. 
- Routing plan mostly finalized, some of the traces are just proof of concept.
those needs to be routed nicely.
Parts:
- added C_sense1: 10nf, Capacitor_SMD:C_0603_1608Metric, symbol AR20_PDM_v1-rescue:C-Device
- added R_sense1: 1k, Resistor_SMD:R_0603_1608Metric, symbol AR20_PDM_v1-rescue:R-Device
Connections:
- net GND: now also C_sense1.1, R_sense1.2
- net MOS_SENSE_ALL: now also C_sense1.2, R_sense1.1
Other:
- note added: "Place relativly close to mcu"
- note added: "Shared sensing circuit for mosfets."
- moved on the sheet: U1

Commit message: First Complete Draft of PCB and schematics, - minus see discription
- missing correct smd switch header
- missing correct main power plug
- tweeks still needs to be done
- Extra inspection of schematics pending
- proper, in depth quiality controll of pcb work pending
Connections:
- net ACM_Shutdown_Circuit: now also U1.1 (14/A0-PC0)
- net CAN_HIGH: now also J2.34
- net CAN_LOW: now also J2.33
- net FP_ENABLE_ACM: no longer U1.22 (4-PD4)
- net FP_ENABLE_AUX: now also J2.3
- net FP_ENABLE_RELAY_SINK: now also J2.30
- net GND: no longer U1.19 (GND), U1.21 (GND), U1.9 (GND)
- net MOS_SENSE_ALL: now also U1.5 (ADC7); no longer U1.1 (14/A0-PC0)
- net P1_EN_ACM: now also U1.22 (4-PD4); no longer U1.20 (3-PD3)
- net P1_OUT: now also J2.1
- net P2_OUT: now also J2.2
- net P3_OUT: now also J2.4
- net P4_OUT: now also J2.5
- net P5_OUT: now also J2.6
- net P6_GearA_open_drain_output: now also J2.14
- net P6_OUT: now also J2.7
- net P7_OUT: now also J2.8
- net RX: now also J2.26
- net SHUTDOWN_IN: now also J2.25; no longer J2.14
- net Switch: now also U1.20 (3-PD3)
- net TX: now also J2.15
- no-connect marks 4 -> 12
Changed lines of the file:
@@
 Text GLabel 8350 950  0    50   Input ~ 0
 vcc_5v
-$Sheet
-S 8475 1650 1500 525
-U 5DE4D361
-F0 "Fuses_Direct" 50
-F1 "Fuses_Direct.sch" 50
-F2 "vcc_5v" I L 8475 1800 50
-F3 "DIRECT_SLC" I L 8475 2025 50
-F4 "DIRECT_SDA" B L 8475 1925 50
-F5 "DIRECT_Alert" O L 8475 2125 50
-F6 "V+12V" I L 8475 1700 50
-F7 "CLUTCH_ACT_OUT" O R 9975 1700 50
-F8 "ETC_OUT" O R 9975 1800 50
-F9 "SHUTDOWN_OUT" O R 9975 1900 50
-F10 "ING_SWITCH_OUT" O R 9975 2000 50
-F11 "MCU_UNITS_FEED_OUT" O R 9975 2100 50
-$EndSheet
 Wire Wire Line
 	2225 875  2125 875
@@
 Text Notes 3350 6950 0    50   ~ 0
 Bulk decoupling cappacitors, place somwhere
-Text HLabel 2925 7075 0    50   Input ~ 10
-V+12V
 Wire Notes Line
 	5900 6750 2500 6750
@@
 Text GLabel 8375 1925 0    50   Input ~ 0
 SDA
-Text GLabel 8375 2125 0    50   Input ~ 0
-DIRECT_Alert
-Wire Wire Line
-	8375 2125 8475 2125
 Text GLabel 10100 750  2    50   Input ~ 0
 COIL_INJECTOR_OUT
@@
 Text GLabel 8350 5300 0    50   Input ~ 0
 P1_MOS_SENSE
-Text GLabel 15175 1725 2    50   Input ~ 0
+Text GLabel 10050 3850 2    50   Input ~ 0
 FP_ENABLE_ACM
 Text GLabel 4375 700  0    50   Input ~ 0
@@
 Text GLabel 8350 5700 0    50   Input ~ 0
 P5_MOS_SENSE
-Text GLabel 8350 5400 0    50   Input ~ 0
+Text GLabel 8350 5600 0    50   Input ~ 0
 P4_MOS_SENSE
 Text GLabel 8350 5500 0    50   Input ~ 0
 P3_MOS_SENSE
-Text GLabel 8350 5600 0    50   Input ~ 0
+Text GLabel 8350 5400 0    50   Input ~ 0
 P2_MOS_SENSE
 $Sheet
@@
 F10 "SDA" I R 10050 4050 50
 F11 "VCC_5v" I R 10050 4175 50
-F12 "EXPANDER_INT" I R 10050 3750 50
-F13 "COIL_INJECTOR_Fault" I L 8225 3075 50
-F14 "FUEL_PUMP_Fault" I L 8225 3175 50
-F15 "P7_Fault" I L 8225 3275 50
-F16 "P6_Fault" I L 8225 3375 50
-F17 "P5_Fault" I L 8225 3475 50
-F18 "P4_Fault" I L 8225 3575 50
-F19 "P3_Fault" I L 8225 3675 50
-F20 "P2_Fault" I L 8225 3775 50
-F21 "P1_Fault" I L 8225 3875 50
+F12 "COIL_INJECTOR_Fault" I L 8225 3075 50
+F13 "FUEL_PUMP_Fault" I L 8225 3175 50
+F14 "P7_Fault" I L 8225 3275 50
+F15 "P6_Fault" I L 8225 3375 50
+F16 "P5_Fault" I L 8225 3475 50
+F17 "P4_Fault" I L 8225 3575 50
+F18 "P3_Fault" I L 8225 3675 50
+F19 "P2_Fault" I L 8225 3775 50
+F20 "P1_Fault" I L 8225 3875 50
+F21 "FP_Alert" I L 8225 4025 50
+F22 "COIL_INJECTOR_Alert" I L 8225 4125 50
+F23 "FP_ENABLE_ACM" O R 10050 3850 50
 $EndSheet
 Text GLabel 10050 4175 2    50   Input ~ 0
@@
 Text GLabel 8225 3075 0    50   Input ~ 0
 COIL_INJECTOR_Fault
-Text GLabel 10050 3750 2    50   Input ~ 0
-EXPANDER_INT
 $Comp
 L AR20_PDM_v1-rescue:GND-power #PWR?
@@
 	0    1    1    0
 $EndComp
-Text HLabel 6825 6825 1    50   Input ~ 10
-V+12V
 $Comp
 L AR20_PDM_v1-rescue:GND-power #PWR?
@@
 	0    1    1    0
 $EndComp
-Text HLabel 7275 6825 1    50   Input ~ 10
-V+12V
 Text Notes 6475 7800 0    50   ~ 0
 Loss of power, flyback protection. \nPlace relativly near all of the mosfets.
 Wire Wire Line
 	11775 7675 11775 7875
-Text GLabel 14050 6825 1    50   Input ~ 0
+Text GLabel 8975 7875 1    50   Input ~ 0
 CAN_LOW
-Text GLabel 13950 6825 1    50   Input ~ 0
+Text GLabel 8875 7875 1    50   Input ~ 0
 CAN_HIGH
 Text GLabel 9375 7875 1    50   Input ~ 0
@@
 Text GLabel 10575 7875 1    50   Input ~ 0
 P7_EN_AUX
-Text GLabel 12125 6775 1    50   Input ~ 0
+Text GLabel 12375 7875 1    50   Input ~ 0
 FP_ENABLE_AUX
 Text GLabel 11675 7875 1    50   Input ~ 0
@@
 Text GLabel 11175 7875 1    50   Input ~ 0
 COIL_INJECTOR_OUT
-Text GLabel 13300 7750 1    50   Input ~ 0
+Text GLabel 12575 7875 1    50   Input ~ 0
 P1_OUT
-Text GLabel 13400 7750 1    50   Input ~ 0
+Text GLabel 12475 7875 1    50   Input ~ 0
 P2_OUT
-Text GLabel 13500 7750 1    50   Input ~ 0
+Text GLabel 12275 7875 1    50   Input ~ 0
 P3_OUT
-Text GLabel 13600 7750 1    50   Input ~ 0
+Text GLabel 12175 7875 1    50   Input ~ 0
 P4_OUT
-Text GLabel 13700 7750 1    50   Input ~ 0
+Text GLabel 12075 7875 1    50   Input ~ 0
 P5_OUT
-Text GLabel 13800 7750 1    50   Input ~ 0
+Text GLabel 11975 7875 1    50   Input ~ 0
 P6_OUT
-Text GLabel 13900 7750 1    50   Input ~ 0
+Text GLabel 11875 7875 1    50   Input ~ 0
 P7_OUT
 $Comp
@@
 $Comp
 L AR20_PDM_v1-rescue:GND-power #PWR?
-U 1 1 5E235210
-P 15175 1275
-AR Path="/5DA89415/5E235210" Ref="#PWR?"  Part="1"
-AR Path="/5DA8920B/5E235210" Ref="#PWR?"  Part="1"
-AR Path="/5DE4D361/5E235210" Ref="#PWR?"  Part="1"
-AR Path="/5E235210" Ref="#PWR012"  Part="1"
-F 0 "#PWR012" H 15175 1025 50  0001 C CNN
-F 1 "GND" V 15175 1075 50  0000 C CNN
-F 2 "" H 15175 1275 50  0001 C CNN
-F 3 "" H 15175 1275 50  0001 C CNN
-	1    15175 1275
-	0    -1   -1   0
-$EndComp
-$Comp
-L AR20_PDM_v1-rescue:GND-power #PWR?
 U 1 1 5E2382FC
 P 15175 1125
@@
 	1    15175 825
 	0    -1   -1   0
-$EndComp
-$Comp
-L AR20_PDM_v1-rescue:GND-power #PWR?
-U 1 1 5E2447FB
-P 15175 1575
-AR Path="/5DA89415/5E2447FB" Ref="#PWR?"  Part="1"
-AR Path="/5DA8920B/5E2447FB" Ref="#PWR?"  Part="1"
-AR Path="/5DE4D361/5E2447FB" Ref="#PWR?"  Part="1"
-AR Path="/5E2447FB" Ref="#PWR013"  Part="1"
-F 0 "#PWR013" H 15175 1325 50  0001 C CNN
-F 1 "GND" V 15175 1375 50  0000 C CNN
-F 2 "" H 15175 1575 50  0001 C CNN
-F 3 "" H 15175 1575 50  0001 C CNN
-	1    15175 1575
-	0    -1   -1   0
-$EndComp
-$Comp
-L AR20_PDM_v1-rescue:GND-power #PWR?
-U 1 1 5E247E0A
-P 13625 2025
-AR Path="/5DA89415/5E247E0A" Ref="#PWR?"  Part="1"
-AR Path="/5DA8920B/5E247E0A" Ref="#PWR?"  Part="1"
-AR Path="/5DE4D361/5E247E0A" Ref="#PWR?"  Part="1"
-AR Path="/5E247E0A" Ref="#PWR08"  Part="1"
-F 0 "#PWR08" H 13625 1775 50  0001 C CNN
-F 1 "GND" V 13625 1825 50  0000 C CNN
-F 2 "" H 13625 2025 50  0001 C CNN
-F 3 "" H 13625 2025 50  0001 C CNN
-	1    13625 2025
-	0    1    1    0
 $EndComp
 Text GLabel 15175 2025 2    50   Input ~ 0
@@
 Text GLabel 15175 2175 2    50   Input ~ 0
 P2_EN_ACM
-Text GLabel 15175 1425 2    50   Input ~ 0
-P1_EN_ACM
 Wire Wire Line
 	2925 7075 3025 7075
@@
 	-1   0    0    1
 $EndComp
-Text GLabel 14450 6825 1    50   Input ~ 0
+Text GLabel 9675 7875 1    50   Input ~ 0
 RX
-Text GLabel 14550 6825 1    50   Input ~ 0
+Text GLabel 10975 7875 1    50   Input ~ 0
 TX
-Text GLabel 14650 6825 1    50   Input ~ 0
+Text GLabel 11075 7875 1    50   Input ~ 0
 P6_GearA_open_drain_output
-Text GLabel 11075 7875 1    50   Input ~ 0
+Text GLabel 9775 7875 1    50   Input ~ 0
 SHUTDOWN_IN
 $Comp
@@
 Wire Wire Line
 	10100 1275 10000 1275
-Text GLabel 12375 3300 0    50   Input ~ 0
+Text GLabel 13625 825  0    50   Input ~ 0
 ACM_Shutdown_Circuit
 NoConn ~ 13625 2325
@@
 F15 "SHUTDOWN_Led" O R 10000 1375 50
 $EndSheet
-Text GLabel 11875 6850 1    50   Input ~ 0
+Text GLabel 9275 7875 1    50   Input ~ 0
 FP_ENABLE_RELAY_SINK
 Wire Wire Line
@@
 Text GLabel 13625 975  0    50   Input ~ 0
 P6_EN_ACM
-Wire Wire Line
-	13650 825  13625 825
-Wire Wire Line
-	12725 825  12725 1500
-Connection ~ 13625 825
-Wire Wire Line
-	13625 825  12725 825
-Wire Wire Line
-	12325 1500 12725 1500
 Text Notes 11575 1975 0    50   ~ 0
 Place relativly close to mcu
@@
 Wire Notes Line
 	11250 675  12925 675
+Wire Wire Line
+	13375 1500 13375 1425
+Wire Wire Line
+	13375 1425 13625 1425
+Wire Wire Line
+	12325 1500 13375 1500
+Text GLabel 8225 4025 0    50   Input ~ 0
+FP_Alert
+Text GLabel 8225 4125 0    50   Input ~ 0
+COIL_INJECTOR_Alert
+NoConn ~ 13625 1725
+Text GLabel 15175 1425 2    50   Input ~ 0
+Switch
+Text GLabel 15175 1725 2    50   Input ~ 0
+P1_EN_ACM
+Text GLabel 2925 7075 0    50   Input ~ 0
+V+12V
+Text GLabel 6825 6825 1    50   Input ~ 0
+V+12V
+Text GLabel 7275 6825 1    50   Input ~ 0
+V+12V
+$Sheet
+S 8475 1650 1500 525
+U 5DE4D361
+F0 "Fuses_Direct" 50
+F1 "Fuses_Direct.sch" 50
+F2 "vcc_5v" I L 8475 1800 50
+F3 "DIRECT_SLC" I L 8475 2025 50
+F4 "DIRECT_SDA" B L 8475 1925 50
+F5 "DIRECT_Alert" O L 8475 2125 50
+F6 "V+12V" I L 8475 1700 50
+F7 "CLUTCH_ACT_OUT" O R 9975 1700 50
+F8 "ETC_OUT" O R 9975 1800 50
+F9 "SHUTDOWN_OUT" O R 9975 1900 50
+F10 "ING_SWITCH_OUT" O R 9975 2000 50
+F11 "MCU_UNITS_FEED_OUT" O R 9975 2100 50
+$EndSheet
+Wire Wire Line
+	8375 2125 8475 2125
+NoConn ~ 8375 2125
+NoConn ~ 13625 2025
+NoConn ~ 9175 7875
+NoConn ~ 9075 7875
+NoConn ~ 15175 1275
+NoConn ~ 15175 1575
+NoConn ~ 1000 6700
 $EndSCHEMATC
