File: AR20_PDM/PDM_schematic/AR_PDM_v1/Misc.sch (KiCad schematic (older format))
At the start: 92 parts, among them P1 B4B-PH-SM4-TB, SW1 SW_DIP_x07, U10 Fet-P, U11 Fet-P, U12 Fet-P, U13 Fet-P, U14 Fet-P, U15 Fet-P, U16 Fet-P, U17 Fet-P, U18 Fet-P, U19 Fet-P, U20 Fet-P, U21 Fet-P, U22 Fet-P, U23 Fet-P, U24 Fet-P, U25 Fet-P, U26 Fet-P, U27 Fet-P, U28 Fet-P

Commit message: Major redesign. schematics completed, PCB work in progress
-TODO : A proper changelog file. Where all changes will apear 
- Redesigned schematics to accommodate errors in the improvement list
- More detail in ALPHA improvement list
Parts:
- removed R42, R43, R48, R49, R56, R57, R62, R63, R65, R66, R69, R70, R72, R73: 4k7, Resistor_SMD:R_0603_1608Metric, symbol AR20_PDM_v1-rescue:R-Device
- removed SW1: SW_DIP_x07, AR_PDM_v1:DIPSwitch, symbol Switch:SW_DIP_x07
- removed U10, U11, U12, U13, U14, U15, U16, U17, U18, U19, U20, U21, U22, U23, U24, U25, U26, U27, U28: Fet-P, Package_TO_SOT_SMD:SOT-23, symbol AR20_PDM_v1-rescue:GenericFet-P
Connections:
- net labels removed: P1_EN_ACM, P1_EN_AUX, P1_MOS_IN, P2_EN_ACM, P2_EN_AUX, P2_MOS_IN, P3_EN_ACM, P3_EN_AUX, P3_MOS_IN, P4_EN_ACM, P4_EN_AUX, P4_MOS_IN, P5_EN_ACM, P5_EN_AUX, P5_MOS_IN, P6_EN_ACM, P6_EN_AUX, P6_MOS_IN, P7_EN_ACM, P7_EN_AUX, P7_MOS_IN
- wire segments 113 -> 29
Other:
- note added: "Load before source !!!!! Redesign"
- note added: "Replece all MOS SYMBOLS !!!\n"
- note removed: "Blown Fuse Detection, for regular fuses. RED-LEDS"
- note removed: "Mosfet controll for ACM"
- note removed: "Mosfet controll for AUX"
- note removed: "Switch for resetting faults on digital phases\nturning ON or OFF each of the mosfets'\nFYI, this switch is multi purpose."
- note removed: "Use Logic Level Mosfets. \n(Gs Threshold <3.3V)\nP-mos array might be used"
- moved on the sheet: D10, D11, D12, D13, D14, D15, D16, D17, D18, D19, D20, D21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
