File: AR20_PDM/PDM_schematic/AR_PDM_v1/backup/AR20_PDM_v1_Back.kicad_pcb (KiCad board)
At the start: 2 copper layers, 110 x 110 mm, 240 parts, among them J1 High_Curret_terminal, J2 1-776163-1, K1 DIPxx-1Cxx-51x, K2 DIPxx-1Cxx-51x, Q1 BTS50025-1TAD, Q10 N_FET, Q11 N_FET, Q12 N_FET, Q13 N_FET, Q14 N_FET, Q15 N_FET, Q16 N_FET, Q17 N_FET, Q2 BTS50025-1TAD, Q3 BTS50025-1TAD, Q4 BTS50025-1TAD, Q5 BTS50025-1TAD, Q6 BTS50025-1TAD, Q7 BTS50025-1TAD, Q8 N_FET, Q9 N_FET, SW1 SW_DIP_x07, SW2 SW_Push, U1 ACM_2020, U10 INA233, U11 INA233, U12 TCA6416A-PortExpander, U13 Fet-P, U14 Fet-P, U15 Fet-P, U16 Fet-P, U17 Fet-P, U18 Fet-P, U19 Fet-P, U2 INA233, U20 Fet-P, U21 Fet-P, U22 Fet-P, U23 Fet-P, U24 Fet-P, U25 Fet-P, U26 Fet-P, U27 Fet-P, U28 Fet-P, U29 Fet-P, U3 INA233, U30 Fet-P, U31 Fet-P, U4 INA233, U5 INA233, U6 INA233, U7 INA233, U8 INA233, U9 INA233

Commit message: PCB design, and issue fixing, work in progress
- Error fixed: Mux mosfet resistor change to ground
- Open drain output added on phase 6, for engine blipping purpose
- Most of pcb symbols and footprints are finished, including main connector
- PCB is change from 1oz to 2oz copper layer, for easier routing.
- Basic Draft of pcb is done, for now.
Parts:
- removed J2: 1-776163-1, AR_PDM_v1:TE_1-776163-1
- removed Q17: N_FET, Package_TO_SOT_SMD:SOT-23
- removed R58: 4K7, Resistor_SMD:R_0603_1608Metric
- removed R_Shunt11: 2m_1%_4W, Resistor_SMD:R_2512_6332Metric
- C10, C13, C14, C9, C_vs1, C_vs2, C_vs3, C_vs4, C_vs5, Cs1, Cs2, Cs3, Cs4, Cs5, R13, R6, R_Shunt1, R_Shunt2, R_s1, R_s2, R_s3, R_s4, R_s5: moved to F.Cu
- C11, C15, C_bypass4, C_bypass5, C_bypass6, C_bypass7, C_bypass8, U10, U11, U5, U6, U7, U8, U9: moved to B.Cu
- moved D28 297.3 mm to (-59.6, 108.6)
- moved D22 284.4 mm to (-54.0, 108.6)
- moved R52 275.9 mm to (-35.8, 114.6)
- moved D20 273.8 mm to (-36.1, 92.1)
- moved D12 271.4 mm to (-48.3, 109.5)
- moved SW1 270.2 mm to (-53.5, 92.4), turned to 0 degrees
- moved D7 265.2 mm to (-59.6, 105.2)
- moved D8 262.8 mm to (-48.3, 106.2)
- moved D10 253.6 mm to (-24.8, 88.7)
- moved D9 253.2 mm to (-54.0, 105.2)
- moved R33 251.3 mm to (-12.2, 95.8)
- moved R39 250.5 mm to (-21.1, 104.4)
- moved D29 250.4 mm to (-30.4, 88.7)
- moved R19 246.3 mm to (-13.0, 103.3)
- moved R47 245.7 mm to (-35.8, 117.1)
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Connections:
- R_s10 pad 1: GND -> MOS_SENSE_ALL
- R_s11 pad 1: GND -> MOS_SENSE_ALL
- R_s12 pad 1: GND -> MOS_SENSE_ALL
- R_s6 pad 1: GND -> MOS_SENSE_ALL
- R_s7 pad 1: GND -> MOS_SENSE_ALL
- R_s8 pad 1: GND -> MOS_SENSE_ALL
- R_s9 pad 1: GND -> MOS_SENSE_ALL
Routing:
- net GND: track 171.7 -> 32.3 mm, vias 16 -> 7
- net SHUTDOWN_OUT: track 50.7 -> 0.00 mm
- net IGN_SWITCH_OUT: track 43.9 -> 0.00 mm
- net CLUTCH_ACT_OUT: track 37.4 -> 0.00 mm
- net ETC_OUT: track 31.1 -> 0.00 mm
- net MCU_UNITS_FEED_OUT: track 23.9 -> 0.00 mm
- net V+12V: track 23.1 -> 0.00 mm, vias 7 -> 0
- net Net-(D3-Pad2): track 18.0 -> 0.00 mm
- net Net-(D1-Pad2): track 17.0 -> 0.00 mm
- net Net-(F_FP1-Pad2): track 13.5 -> 0.00 mm
- net Net-(F_COIL1-Pad2): track 6.08 -> 0.00 mm
- net P6_MOS_SENSE: track 3.31 -> 0.00 mm, vias 1 -> 0
- net P5_MOS_SENSE: track 3.31 -> 0.00 mm, vias 1 -> 0
- net P4_MOS_SENSE: track 3.31 -> 0.00 mm, vias 1 -> 0
- net P3_MOS_SENSE: track 3.31 -> 0.00 mm, vias 1 -> 0
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- removed copper zone on F.Cu, net V+12V
Other:
- board size 110 x 110 mm -> 120 x 120 mm
- net class Default: clearance 0.127 -> 0.2
- rule trace_clearance: 0.127 -> 0.2
